File: 1v8_buck.kicad_sch (KiCad schematic)
At the start: 0 parts

Commit message: power scheme
Parts:
- added C901, C902: 10uF 10V, BR_Passives:C_0402_1005Metric-minimized, symbol BR_Capacitors_0402:C_0402_10uF_10V_X5R_20%
- added L901: 2u2 2.2A, BR_Inductors:L_Taiyo-Yuden_NR-4018, symbol BR_Inductors:L_NRS4018T2R2MDGJV
- added NT901: NetTie-2_0.18mm, BR_Virtual_Parts:NetTie-2_SMD_Pad_0.18mm_wide_long, symbol BR_Virtual_Parts:NetTie-2_0.18mm_long
- added R901: 10k, BR_Passives:R_0201_0603Metric-minimized, symbol BR_Resistors_0201:R_0201_10k
- added U901: TLV62569DBVR, BR_SOT:SOT-23-5_mini, symbol BR_IC_Regulators:TLV62569DBVR
Connections:
- new net EN: U901.1 (EN)
- new net GND: NT901.2, R901.2
- new net PGND: C901.2, C902.2, NT901.1, U901.2 (GND)
- new net RSET: R901.1, U901.5 (FB)
- new net SW: L901.1, U901.3 (SW)
- new net VIN: C901.1, U901.4 (VIN)
- new net VOUT: C902.1, L901.2
Other:
- note added: "5V or 3.3V"
- note added: "Controlled to 0.6V"
- note added: "DeltaIL = Vout * (1-Vout/Vin)/(L*Fsw) = 0.33A for 5-3.3V = 0.67A for 3.3-1.1V"
- note added: "Fsw = 1.5MHz"
- note added: "High-side current limit is 3A. Switches to low side for protection"
- note added: "IL(max) = Iout + DeltaIL/2 Iout = IL(max) - DeltaIL/2 = 2.67A (5-3.3V) = 2.84A (3.3-1.1V) Both near sat. of inductor"
- note added: "Max 6V"
- note added: "Saturation current is 3A"
