File: 4v5_buck.kicad_sch (KiCad schematic)
At the start: 0 parts

Commit message: power scheme
Parts:
- added U3: MIC28517T-E/PHA, BR_IC:QFN-32_x6mm_P0.65mm, symbol BR_IC_Regulators:MIC28517T-E/PHA
Connections:
- new net: U3.12 (SW), U3.13 (SW), U3.14 (SW), U3.15 (SW)
- new net PGND: U3.16 (PGND), U3.17 (PGND), U3.18 (PGND), U3.19 (PGND)
- new net PVIN: U3.10 (PVIN), U3.11 (PVIN), U3.5 (PVIN), U3.6 (PVIN), U3.7 (PVIN), U3.8 (PVIN), U3.9 (PVIN)
Changed lines of the file:
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@@
 	(generator_version "9.0")
 	(paper "A4")
+	(symbol
+		(lib_id "BR_IC_Regulators:MIC28517T-E/PHA")
+		(at 147.32 76.2 0)
+		(unit 1)
+		(exclude_from_sim no)
+		(in_bom yes)
+		(on_board yes)
+		(dnp no)
+		(fields_autoplaced yes)
+		(property "Reference" "U3"
+			(at 147.32 58.42 0)
+			(effects
+				(font
+					(size 1.27 1.27)
+				)
+			)
+		)
+		(property "Value" "MIC28517T-E/PHA"
+			(at 147.32 60.96 0)
+			(effects
+				(font
+					(size 1.27 1.27)
+				)
+			)
+		)
+		(property "Footprint" "BR_IC:QFN-32_x6mm_P0.65mm"
+			(at 147.32 0 0)
+			(effects
+				(font
+					(size 1.27 1.27)
+				)
+				(justify left)
+				(hide yes)
+			)
+		)
+		(property "Datasheet" "https://ww1.microchip.com/downloads/aemDocuments/documents/APID/ProductDocuments/DataSheets/MIC28517-Data-Sheet-DS20006317C.pdf"
+			(at 147.32 2.54 0)
+			(effects
+				(font
+					(size 1.27 1.27)
+				)
+				(justify left)
+				(hide yes)
+			)
+		)
+		(property "Description" "Buck Switching Regulator, Adjustable, 8A, 600mV~32V, 4.5V~70V, VQFN-32(6x6)"
+			(at 147.32 5.08 0)
+			(effects
+				(font
+					(size 1.27 1.27)
+				)
+				(justify left)
+				(hide yes)
+			)
+		)
+		(property "Manufacturer" "Microchip Technology"
+			(at 147.32 7.62 0)
+			(effects
+				(font
+					(size 1.27 1.27)
+				)
+				(justify left)
+				(hide yes)
+			)
+		)
+		(property "Manufacturer Part Num" "MIC28517T-E/PHA"
+			(at 147.32 10.16 0)
+			(effects
+				(font
+					(size 1.27 1.27)
+				)
+				(justify left)
+				(hide yes)
+			)
+		)
+		(property "BRE Number" "BRE-001217"
+			(at 147.32 12.7 0)
+			(effects
+				(font
+					(size 1.27 1.27)
+				)
+				(justify left)
+				(hide yes)
+			)
+		)
+		(property "Supplier 1" "DigiKey"
+			(at 147.32 15.24 0)
+			(effects
+				(font
+					(size 1.27 1.27)
+				)
+				(justify left)
+				(hide yes)
+			)
+		)
+		(property "Supplier Part Num 1" "150-MIC28517T-E/PHACT-ND"
+			(at 147.32 17.78 0)
+			(effects
+				(font
+					(size 1.27 1.27)
+				)
+				(justify left)
+				(hide yes)
+			)
+		)
+		(property "Supplier 2" "Mouser"
+			(at 147.32 20.32 0)
+			(effects
+				(font
+					(size 1.27 1.27)
+				)
+				(justify left)
+				(hide yes)
+			)
+		)
+		(property "Supplier Part Num 2" "579-MIC28517T-E/PHA"
+			(at 147.32 22.86 0)
+			(effects
+				(font
+					(size 1.27 1.27)
+				)
+				(justify left)
+				(hide yes)
+			)
+		)
+		(property "Supplier 3" "JLCPCB"
+			(at 147.32 25.4 0)
+			(effects
+				(font
+					(size 1.27 1.27)
+				)
+				(justify left)
+				(hide yes)
+			)
+		)
+		(property "Supplier Part Num 3" "C623943"
+			(at 147.32 27.94 0)
+			(effects
+				(font
+					(size 1.27 1.27)
+				)
+				(justify left)
+				(hide yes)
+			)
+		)
+		(property "JLCPCB Part Num" "C623943"
+			(at 147.32 30.48 0)
+			(effects
+				(font
+					(size 1.27 1.27)
+				)
+				(justify left)
+				(hide yes)
+			)
+		)
+		(pin "2"
+		)
+		(pin "3"
+		)
+		(pin "21"
+		)
+		(pin "19"
+		)
+		(pin "30"
+		)
+		(pin "16"
+		)
+		(pin "17"
+		)
+		(pin "7"
+		)
+		(pin "18"
+		)
+		(pin "22"
+		)
+		(pin "29"
+		)
+		(pin "32"
+		)
+		(pin "24"
+		)
+		(pin "33"
+		)
+		(pin "4"
+		)
+		(pin "25"
+		)
+		(pin "20"
+		)
+		(pin "15"
+		)
+		(pin "9"
+		)
+		(pin "8"
+		)
+		(pin "26"
+		)
+		(pin "28"
+		)
+		(pin "13"
+		)
+		(pin "1"
+		)
+		(pin "12"
+		)
+		(pin "23"
+		)
+		(pin "14"
+		)
+		(pin "27"
+		)
+		(pin "31"
+		)
+		(pin "5"
+		)
+		(pin "6"
+		)
+		(pin "10"
+		)
+		(pin "11"
+		)
+		(instances
+			(project ""
+				(path "/2a5ce3ef-537a-4122-a1be-ef76186bc0d7/774f2c6c-c15c-4713-acf0-4edb2ec6be20/623c30ef-7a3a-4d24-b1c0-70fa5da5cbd0"
+					(reference "U3")
+					(unit 1)
+				)
+			)
+		)
+	)
 )
