File: SonarDevBoard.kicad_pcb (KiCad board)
At the start: 2 copper layers, 83 parts, among them U5 LM5160ADNTR, U6 STM32H563AII3Q, X1 25MHz 8pF

Commit message: updates
Parts:
- added C61: 10uF 100V, BR_Passives:C_1210_3225Metric, F.Cu at (66.8, 19.9)
- added C7: 100nF 25V, BR_Passives:C_0201_0603Metric-minimized, F.Cu at (66.7, 59.4)
- added D2: 10V, BR_Discretes:D_SOD-323, F.Cu at (66.3, 23.2)
- added H1: M3_Clearance_Plated_6mm, BR_Virtual_Parts:M3_Clearance_Plated_6mm, F.Cu at (145.0, 89.5)
- added H2: M3_Clearance_Plated_6mm, BR_Virtual_Parts:M3_Clearance_Plated_6mm, F.Cu at (45.0, 89.5)
- added H3: M3_Clearance_Plated_6mm, BR_Virtual_Parts:M3_Clearance_Plated_6mm, F.Cu at (45.0, 139.5)
- added H4: M3_Clearance_Plated_6mm, BR_Virtual_Parts:M3_Clearance_Plated_6mm, F.Cu at (145.0, 139.5)
- added J1: POWER, BR_Connectors_JST:BM02B-GHS-TBT, F.Cu at (60.7, 21.7)
- added J2: ETHERNET, BR_Connectors_JST:BM04B-GHS-TBT, F.Cu at (61.9, 34.8)
- added J3: TRANSDUCER, BR_Connectors_JST:BM02B-GHS-TBT, F.Cu at (60.7, 28.3)
- added Q1: DMP6023LSS-13, BR_SO:SO-8_3.9x4.9mm_P1.27mm, F.Cu at (61.3, 41.0)
- added Q2: MJD44H11T4G, BR_SOT:TO-252-2_L6.5-W6.1-P4.58-LS10.0-TL, F.Cu at (40.4, 22.0)
- added Q3: MJD45H11T4G, BR_SOT:TO-252-2_L6.5-W6.1-P4.58-LS10.0-TL, F.Cu at (40.4, 30.0)
- added Q4: MJD45H11T4G, BR_SOT:TO-252-2_L6.5-W6.1-P4.58-LS10.0-TL, F.Cu at (40.4, 38.0)
- added Q5: MJD44H11T4G, BR_SOT:TO-252-2_L6.5-W6.1-P4.58-LS10.0-TL, F.Cu at (40.4, 46.0)
- added R15: 47k, BR_Passives:R_0201_0603Metric-minimized, F.Cu at (66.7, 61.0)
- added R18: 3k, BR_Passives:R_0201_0603Metric-minimized, F.Cu at (66.7, 62.5)
- added R36: 47k, BR_Passives:R_0201_0603Metric-minimized, F.Cu at (65.4, 25.4)
- added T1: HR641680E, BR_Inductors:H1102FNL, F.Cu at (56.7, 54.9)
- added TP35: TP_ROUND_TH_300um, BR_Virtual_Parts:TP_ROUND_SMT_300um, F.Cu at (66.4, 49.9)
- added TP36: TP_ROUND_TH_300um, BR_Virtual_Parts:TP_ROUND_SMT_300um, F.Cu at (66.4, 51.4)
- added TP40: TP_ROUND_TH_300um, BR_Virtual_Parts:TP_ROUND_SMT_300um, F.Cu at (66.4, 52.9)
- added TP41: TP_ROUND_TH_300um, BR_Virtual_Parts:TP_ROUND_SMT_300um, F.Cu at (66.4, 54.4)
- added TP42: TP_ROUND_TH_300um, BR_Virtual_Parts:TP_ROUND_SMT_300um, F.Cu at (66.4, 55.9)
- added TP43: TP_ROUND_TH_300um, BR_Virtual_Parts:TP_ROUND_SMT_300um, F.Cu at (67.9, 49.9)
- added TP44: TP_ROUND_TH_300um, BR_Virtual_Parts:TP_ROUND_SMT_300um, F.Cu at (67.9, 51.4)
- added TP45: TP_ROUND_TH_300um, BR_Virtual_Parts:TP_ROUND_SMT_300um, F.Cu at (67.9, 52.9)
- added TP46: TP_ROUND_TH_300um, BR_Virtual_Parts:TP_ROUND_SMT_300um, F.Cu at (67.9, 54.4)
- added TP47: TP_ROUND_TH_300um, BR_Virtual_Parts:TP_ROUND_SMT_300um, F.Cu at (67.9, 55.9)
- added TP48: TP_ROUND_TH_300um, BR_Virtual_Parts:TP_ROUND_SMT_300um, F.Cu at (69.4, 49.9)
- added TP49: TP_ROUND_TH_300um, BR_Virtual_Parts:TP_ROUND_SMT_300um, F.Cu at (69.4, 51.4)
- added TP50: TP_ROUND_TH_300um, BR_Virtual_Parts:TP_ROUND_SMT_300um, F.Cu at (69.4, 52.9)
- added U1: DP83825IRMQR, BR_IC:WQFN-24-3x3x0.8mm-DRV8311, F.Cu at (52.2, 63.0)
- added U2: W958D8NBYA5I, BR_IC:BGA-24_6x8mm_Layout5x5_P1.0mm, F.Cu at (39.4, 57.5)
Connections:
- net /3V3 Buck/SW renamed /Power/3V3 Buck/SW
- net /BOOST_MODE renamed /MCU/BOOST_MODE
- net /COMM_N renamed /MCU/COMM_N
- net /COMM_P renamed /MCU/COMM_P
- net /DAC renamed /MCU/DAC
- net /DEBUG_LED renamed /MCU/DEBUG_LED
- net /I2C4.SCL renamed /MCU/I2C4.SCL
- net /I2C4.SDA renamed /MCU/I2C4.SDA
- net /ISENSE renamed /MCU/ISENSE
- net /LED_ENABLE renamed /MCU/LED_ENABLE
- net /MAC.MDC renamed /MCU/MAC.MDC
- net /MAC.MDIO renamed /MCU/MAC.MDIO
- net /MAC.RXD0 renamed /MCU/MAC.RXD0
- net /MAC.RXD1 renamed /MCU/MAC.RXD1
- net /MAC.RXDV renamed /MCU/MAC.RXDV
- net /MAC.RXER renamed /MCU/MAC.RXER
- net /MAC.TXD0 renamed /MCU/MAC.TXD0
- net /MAC.TXD1 renamed /MCU/MAC.TXD1
- net /MAC.TXEN renamed /MCU/MAC.TXEN
- net /OSC_IN renamed /MCU/OSC_IN
- net /OSC_OUT renamed /MCU/OSC_OUT
- net /PHY_GPIO0 renamed /MCU/PHY_GPIO0
- net /PHY_INH renamed /MCU/PHY_INH
- net /PHY_REF_CLK renamed /MCU/PHY_REF_CLK
- net /PHY_WAKE_IN renamed /MCU/PHY_WAKE_IN
- net /PHY_WAKE_OUT renamed /MCU/PHY_WAKE_OUT
- net /PHY_nIRQ renamed /MCU/PHY_nIRQ
- net /PHY_nRST renamed /MCU/PHY_nRST
- net /SWCLK renamed /MCU/SWCLK
- net /SWDIO renamed /MCU/SWDIO
- net /T1S_TERM_GATE renamed /MCU/T1S_TERM_GATE
- net /TIM4_CH1 renamed /MCU/TIM4_CH1
- net /TIM4_CH3 renamed /MCU/TIM4_CH3
- net /USART1.RX renamed /MCU/USART1.RX
- net /USART1.TX renamed /MCU/USART1.TX
- net /VCAP1 renamed /MCU/VCAP1
- net /VCAP2 renamed /MCU/VCAP2
- net /VSENSE renamed /MCU/VSENSE
- net /VTHERM renamed /MCU/VTHERM
- net /nRST renamed /MCU/nRST
- net VIN_PROTECTED renamed /Power/VIN_PROTECTED
- C56 pad 2: 3V3 -> /Power/3V3
- C59 pad 1: 3V3 -> /Power/3V3
- L1 pad 2: 3V3 -> /Power/3V3
- R5 pad 1: 3V3 -> /Power/3V3
- U6 pad C3: unconnected-(U6-PE2-PadC3) -> /MCU/OCTOSPI1.IO2
- U6 pad E6: unconnected-(U6-PB5-PadE6) -> /MCU/OCTOSPI1.NCLK
- U6 pad G2: unconnected-(U6-PF9-PadG2) -> /MCU/OCTOSPI1.IO1
- U6 pad G4: unconnected-(U6-PF8-PadG4) -> /MCU/OCTOSPI1.IO0
- U6 pad G7: unconnected-(U6-PF6-PadG7) -> /MCU/OCTOSPI1.IO3
- U6 pad H4: unconnected-(U6-PF10-PadH4) -> /MCU/OCTOSPI1.CLK
- U6 pad J4: unconnected-(U6-PH2-PadJ4) -> /MCU/OCTOSPI1.IO4
- U6 pad J8: unconnected-(U6-PE8-PadJ8) -> /MCU/OCTOSPI1.IO5
- U6 pad L8: unconnected-(U6-PE10-PadL8) -> /MCU/OCTOSPI1.IO7
- U6 pad M8: unconnected-(U6-PE11-PadM8) -> /MCU/OCTOSPI1.NCS
- U6 pad M9: unconnected-(U6-PE12-PadM9) -> /MCU/PSRAM_nRST
- U6 pad N6: unconnected-(U6-PB2-PadN6) -> /MCU/OCTOSPI1.DQS
- U6 pad N8: unconnected-(U6-PE9-PadN8) -> /MCU/OCTOSPI1.IO6
Other:
- board outline added: 110 x 60 mm

Commit message: power scheme
Parts:
- added C301: 10uF 10V, BR_Passives:C_0402_1005Metric-minimized, F.Cu at (141.0, 38.8)
- added C302: 10uF 10V, BR_Passives:C_0402_1005Metric-minimized, F.Cu at (142.6, 38.8)
- added C901: 10uF 10V, BR_Passives:C_0402_1005Metric-minimized, F.Cu at (153.0, 38.6)
- added C902: 10uF 10V, BR_Passives:C_0402_1005Metric-minimized, F.Cu at (154.6, 38.6)
- added L301: 2u2 2.2A, BR_Inductors:L_Taiyo-Yuden_NR-4018, F.Cu at (146.0, 37.0)
- added L901: 2u2 2.2A, BR_Inductors:L_Taiyo-Yuden_NR-4018, F.Cu at (158.0, 36.9)
- added NT301: NetTie-2_0.18mm, BR_Virtual_Parts:NetTie-2_SMD_Pad_0.18mm_wide_long, F.Cu at (142.7, 36.6)
- added NT901: NetTie-2_0.18mm, BR_Virtual_Parts:NetTie-2_SMD_Pad_0.18mm_wide_long, F.Cu at (154.7, 36.4)
- added R104: 45k3, BR_Passives:R_0201_0603Metric-minimized, B.Cu at (143.0, 38.0)
- added R112: 8k25, BR_Passives:C_0201_0603Metric-minimized, B.Cu at (155.0, 38.2)
- added R301: 10k, BR_Passives:R_0201_0603Metric-minimized, B.Cu at (143.0, 36.8)
- added R901: 10k, BR_Passives:R_0201_0603Metric-minimized, B.Cu at (155.0, 36.7)
- added U301: TLV62569DBVR, BR_SOT:SOT-23-5_mini, F.Cu at (142.0, 36.5)
- added U901: TLV62569DBVR, BR_SOT:SOT-23-5_mini, F.Cu at (154.0, 36.4)
Routing:
- net /3V3 Buck/SW: track 0.00 -> 2.88 mm
- net /1V1 Buck/SW: track 0.00 -> 2.88 mm
- net /3V3 Buck/PGND: track 0.00 -> 0.70 mm
- net /1V1 Buck/PGND: track 0.00 -> 0.70 mm
- net /1V1 Buck/RSET: track 0.00 -> 0.60 mm
- net GND: vias 0 -> 2
- net 3V3: vias 0 -> 1
- net 1V1: vias 0 -> 1
- added copper zone on F.Cu, net /1V1 Buck/PGND
- added copper zone on F.Cu, net /3V3 Buck/PGND
- added copper zone on F.Cu, net 1V1
- added copper zone on F.Cu, net 3V3
- added copper zone on F.Cu, net 5V

Commit message: layout start
Parts:
- removed C20, C56: 10nF 50V, BR_Passives:C_0402_1005Metric-minimized
- removed C22, C5: 2u2F 10V, BR_Passives:C_0402_1005Metric-minimized
- removed C23, C46: 1uF 50V, BR_Passives:C_0402_1005Metric-minimized
- removed the C302 at (142.6, 38.8)
- removed C57: 100nF 25V, BR_Passives:C_0201_0603Metric-minimized
- removed C58: 10uF 100V, BR_Passives:C_1210_3225Metric
- removed C59: 22uF 25V, BR_Passives:C_0805_2012Metric-minimized
- removed J1: POWER, BR_Connectors_JST:BM02B-GHS-TBT
- removed L1: 10uH 2.45A, BR_Inductors:IND_VLS6045EX-101M
- removed L901: 2u2 2.2A, BR_Inductors:L_Taiyo-Yuden_NR-4018
- removed NT2, NT301, NT901: NetTie-2_0.18mm, BR_Virtual_Parts:NetTie-2_SMD_Pad_0.18mm_wide_long
- removed Q2, Q5: MJD44H11T4G, BR_SOT:TO-252-2_L6.5-W6.1-P4.58-LS10.0-TL
- removed Q3, Q4: MJD45H11T4G, BR_SOT:TO-252-2_L6.5-W6.1-P4.58-LS10.0-TL
- removed R21: 30k, BR_Passives:R_0201_0603Metric-minimized
- removed R23, R27: 4k7, BR_Passives:R_0201_0603Metric-minimized
- removed the R301 at (143.0, 36.8)
- removed R38, R6, R8, R901: 10k, BR_Passives:R_0201_0603Metric-minimized
- removed R4: 49k9, BR_Passives:R_0201_0603Metric-minimized
- removed R5: 6k49, BR_Passives:R_0201_0603Metric-minimized
- removed TP1, TP19, TP2, TP20, TP21, TP31, TP32, TP33, TP34, TP38, TP5, TP6: TP_ROUND_TH_300um, BR_Virtual_Parts:TP_ROUND_SMT_300um
- removed the U301 at (142.0, 36.5)
- removed U5: LM5160ADNTR, BR_IC:WSON-12-1EP_4x4mm_P0.5mm_EP2.6x3mm
- removed the U901 at (154.0, 36.4)
- added C1001: 100nF 25V, BR_Passives:C_0201_0603Metric-minimized, F.Cu at (241.9, 80.6)
- added C1002: 100nF 25V, BR_Passives:C_0201_0603Metric-minimized, F.Cu at (241.9, 82.2)
- added C1003: 100nF 100V, BR_Passives:C_0402_1005Metric-minimized, F.Cu at (230.7, 80.8)
- added C1004: 100nF 100V, BR_Passives:C_0402_1005Metric-minimized, F.Cu at (230.7, 82.6)
- added C1005: 4u7F 100V, BR_Passives:C_1206_3216Metric-minimized, F.Cu at (243.9, 94.4)
- added C1006: 100nF 100V, BR_Passives:C_0402_1005Metric-minimized, F.Cu at (230.7, 84.5)
- added C1007: 100nF 100V, BR_Passives:C_0402_1005Metric-minimized, F.Cu at (230.7, 86.3)
- added C1008: 100nF 25V, BR_Passives:C_0201_0603Metric-minimized, F.Cu at (241.9, 83.7)
- added C101: 100nF 50V, BR_Passives:C_0402_1005Metric-minimized, F.Cu at (145.1, 94.0)
- added C102: 2u2F 100V, BR_Passives:C_0805_2012Metric-minimized, F.Cu at (210.8, 50.1)
- added C103: 100nF 50V, BR_Passives:C_0402_1005Metric-minimized, F.Cu at (45.5, 94.0)
- added C104: 100nF 25V, BR_Passives:C_0201_0603Metric-minimized, F.Cu at (204.8, 54.2)
- added C106: 2u2F 100V, BR_Passives:C_0805_2012Metric-minimized, F.Cu at (210.8, 52.7)
- added C107: 100nF 50V, BR_Passives:C_0402_1005Metric-minimized, F.Cu at (44.5, 135.5)
- added C108: 220nF 100V, BR_Passives:C_0603_1608Metric-minimized, F.Cu at (224.1, 49.9)
- added C109: 100nF 50V, BR_Passives:C_0402_1005Metric-minimized, F.Cu at (145.1, 135.0)
- added C110: 220nF 100V, BR_Passives:C_0603_1608Metric-minimized, F.Cu at (224.1, 52.2)
- added C1101: 10uF 10V, BR_Passives:C_0402_1005Metric-minimized, F.Cu at (278.4, 22.2)
- added C1102: 10uF 10V, BR_Passives:C_0402_1005Metric-minimized, F.Cu at (278.4, 24.0)
- added C111: 470nF 100V, BR_Passives:C_0805_2012Metric-minimized, F.Cu at (210.8, 55.3)
- added C112: 470nF 100V, BR_Passives:C_0805_2012Metric-minimized, F.Cu at (210.8, 57.9)
- added C113: 100nF 25V, BR_Passives:C_0201_0603Metric-minimized, F.Cu at (204.8, 55.7)
- added C114: 1uF 50V, BR_Passives:C_0402_1005Metric-minimized, F.Cu at (213.3, 29.5)
- added C1201: 10nF 50V, BR_Passives:C_0402_1005Metric-minimized, F.Cu at (215.8, 65.9)
- added C1202: 10uF 100V, BR_Passives:C_1210_3225Metric, F.Cu at (217.0, 74.3)
- added C1203: 470nF 16V, BR_Passives:C_0402_1005Metric-minimized, F.Cu at (215.8, 67.7)
- added C1204: 100nF 25V, BR_Passives:C_0201_0603Metric-minimized, F.Cu at (219.9, 84.7)
- added C1205: 22nF 50V, BR_Passives:C_0402_1005Metric, F.Cu at (215.9, 91.4)
- added C1206: 1uF 50V, BR_Passives:C_0402_1005Metric-minimized, F.Cu at (215.8, 69.6)
- added C1207: 10uF 16V, BR_Passives:C_0603_1608Metric-minimized, F.Cu at (220.1, 88.7)
- added C1208: 220uF 100V, BR_Passives:C_Elec_12.5x12.5, F.Cu at (194.2, 102.0)
- added C1209: 100nF 100V, BR_Passives:C_0603_1608Metric-minimized, F.Cu at (220.1, 90.9)
- added C1210: 100nF 100V, BR_Passives:C_0603_1608Metric-minimized, F.Cu at (220.1, 93.2)
- added C1211: 10uF 100V, BR_Passives:C_1210_3225Metric, F.Cu at (217.0, 78.1)
- added C1212: 10uF 100V, BR_Passives:C_1210_3225Metric, F.Cu at (217.0, 82.0)
- added C1213: 100nF 50V, BR_Passives:C_0402_1005Metric-minimized, F.Cu at (215.8, 71.4)
- added C1214: 4u7F 10V, BR_Passives:C_0402_1005Metric-minimized, F.Cu at (218.4, 65.9)
- added C1301: 2u2F 10V, BR_Passives:C_0402_1005Metric-minimized, F.Cu at (250.7, 100.1)
- added C1302: 330pF 50V, BR_Passives:C_0402_1005Metric, F.Cu at (253.4, 108.5)
- added C1303: 10uF 10V, BR_Passives:C_0402_1005Metric-minimized, F.Cu at (250.7, 101.9)
- added C1401: 330nF 16V, BR_Passives:C_0402_1005Metric-minimized, F.Cu at (230.7, 107.8)
- added C1402: 100nF 25V, BR_Passives:C_0201_0603Metric-minimized, F.Cu at (233.1, 107.7)
- added C1501: 1uF 10V, BR_Passives:C_0402_1005Metric-minimized, F.Cu at (275.2, 80.8)
- added C1502: 100nF 100V, BR_Passives:C_0603_1608Metric-minimized, F.Cu at (275.6, 90.2)
- added C1503: 100nF 50V, BR_Passives:C_0402_1005Metric-minimized, F.Cu at (275.2, 82.6)
- added C1504: 100nF 50V, BR_Passives:C_0402_1005Metric-minimized, F.Cu at (275.2, 84.5)
- added C1505: 100nF 100V, BR_Passives:C_0603_1608Metric-minimized, F.Cu at (275.6, 92.4)
- added C1506: 1uF 10V, BR_Passives:C_0402_1005Metric-minimized, F.Cu at (275.2, 86.3)
- added C1601: 2u2F 10V, BR_Passives:C_0402_1005Metric-minimized, F.Cu at (272.2, 37.1)
- added C1602: 10nF 50V, BR_Passives:C_0402_1005Metric-minimized, F.Cu at (272.2, 38.9)
- added C1603: 10nF 50V, BR_Passives:C_0402_1005Metric-minimized, F.Cu at (272.2, 40.7)
- added C1604: 220nF 25V, BR_Passives:C_0402_1005Metric-minimized, F.Cu at (272.2, 42.6)
- added C1605: 22nF 50V, BR_Passives:C_0402_1005Metric, F.Cu at (274.9, 48.0)
- added C1606: 1uF 10V, BR_Passives:C_0402_1005Metric-minimized, F.Cu at (272.2, 44.4)
- added C305: 4u7F 6V3, BR_Passives:C_0201_0603Metric-minimized, F.Cu at (265.2, 36.9)
- added C308: 4u7F 6V3, BR_Passives:C_0201_0603Metric-minimized, F.Cu at (265.2, 38.5)
- added C310: 4u7F 6V3, BR_Passives:C_0201_0603Metric-minimized, F.Cu at (265.2, 40.0)
- added C316: 100pF 50V, BR_Passives:C_0201_0603Metric-minimized, F.Cu at (265.2, 41.6)
- added C401: 100nF 100V, BR_Passives:C_0402_1005Metric-minimized, F.Cu at (243.5, 59.7)
- added C402: 200pF 50V, BR_Passives:C_0402_1005Metric, F.Cu at (255.3, 70.1)
- added C403: 1uF 10V, BR_Passives:C_0402_1005Metric-minimized, F.Cu at (243.5, 61.5)
- added C404: 47nF 50V, BR_Passives:C_0402_1005Metric-minimized, F.Cu at (243.5, 63.4)
- added C405: 15nF, BR_Passives:C_0402_1005Metric-minimized, F.Cu at (243.5, 65.2)
- added C406: 15nF, BR_Passives:C_0402_1005Metric-minimized, F.Cu at (243.5, 67.1)
- added C407: 100nF 50V, BR_Passives:C_0402_1005Metric-minimized, F.Cu at (243.5, 68.9)
- added C408: 3.9pF 50V, BR_Passives:C_0402_1005Metric, F.Cu at (255.3, 72.1)
- added C409: 3.9pF 50V, BR_Passives:C_0402_1005Metric, F.Cu at (255.3, 74.1)
- added C410: 1uF 16V, BR_Passives:C_0201_0603Metric-minimized, F.Cu at (248.6, 72.4)
- added C411: 1uF 10V, BR_Passives:C_0402_1005Metric-minimized, F.Cu at (243.5, 70.7)
- added C412: 100nF 50V, BR_Passives:C_0402_1005Metric-minimized, F.Cu at (246.1, 59.7)
- added C601: 100nF 50V, BR_Passives:C_0402_1005Metric-minimized, F.Cu at (259.4, 22.2)
- added C602: 4u7F 10V, BR_Passives:C_0402_1005Metric-minimized, F.Cu at (259.4, 24.0)
- added C603: 4u7F 10V, BR_Passives:C_0402_1005Metric-minimized, F.Cu at (259.4, 25.9)
- added C604: 100nF 50V, BR_Passives:C_0402_1005Metric-minimized, F.Cu at (259.4, 27.7)
- added C605: 330nF 16V, BR_Passives:C_0402_1005Metric-minimized, F.Cu at (259.4, 29.5)
- added C606: 100nF 50V, BR_Passives:C_0402_1005Metric-minimized, F.Cu at (259.4, 31.4)
- added C701: 10uF 10V, BR_Passives:C_0402_1005Metric-minimized, F.Cu at (270.3, 96.5)
- added C702: 1nF 2kV, BR_Passives:C_1206_3216Metric-minimized, F.Cu at (271.4, 104.4)
- added C703: 1uF 10V, BR_Passives:C_0402_1005Metric-minimized, F.Cu at (270.3, 98.3)
- added C704: 100nF 25V, BR_Passives:C_0201_0603Metric-minimized, F.Cu at (267.9, 96.3)
- added C705: 10nF 25V, BR_Passives:C_0201_0603Metric-minimized, F.Cu at (267.9, 97.9)
- added C706: 10nF 25V, BR_Passives:C_0201_0603Metric-minimized, F.Cu at (267.9, 99.4)
- added C707: 100nF 25V, BR_Passives:C_0201_0603Metric-minimized, F.Cu at (267.9, 101.0)
- added C708: 100nF 25V, BR_Passives:C_0201_0603Metric-minimized, F.Cu at (267.9, 102.5)
- added C709: 1uF 10V, BR_Passives:C_0402_1005Metric-minimized, F.Cu at (270.3, 100.2)
- added C710: 1uF 10V, BR_Passives:C_0402_1005Metric-minimized, F.Cu at (270.3, 102.0)
- added C711: 10uF 10V, BR_Passives:C_0402_1005Metric-minimized, F.Cu at (272.9, 96.5)
- added C712: 1nF 2kV, BR_Passives:C_1206_3216Metric-minimized, F.Cu at (271.4, 107.3)
- added C803: 2u2F 100V, BR_Passives:C_0805_2012Metric-minimized, F.Cu at (42.1, 212.2)
- added C804: 2u2F 100V, BR_Passives:C_0805_2012Metric-minimized, F.Cu at (42.1, 214.8)
- added C805: 2u2F 100V, BR_Passives:C_0805_2012Metric-minimized, F.Cu at (42.1, 217.4)
- added C806: 4u7F 10V, BR_Passives:C_0402_1005Metric-minimized, F.Cu at (26.0, 226.0)
- added C807: 1uF 100V, BR_Passives:C_0805_2012Metric-minimized, F.Cu at (42.1, 220.0)
- added C808: 2u2F 10V, BR_Passives:C_0402_1005Metric-minimized, F.Cu at (26.0, 227.9)
- added C809: 100nF 100V, BR_Passives:C_0603_1608Metric-minimized, F.Cu at (42.8, 226.2)
- added C810: 100nF 100V, BR_Passives:C_0402_1005Metric-minimized, F.Cu at (26.0, 229.7)
- added C811: 4n7F 100V, BR_Passives:C_0402_1005Metric, F.Cu at (42.5, 232.8)
- added C812: 10uF 10V, BR_Passives:C_0603_1608Metric-minimized, F.Cu at (42.8, 228.5)
- added C813: 10uF 10V, BR_Passives:C_0603_1608Metric-minimized, F.Cu at (42.8, 230.7)
- added D1201: BAS20H, BR_Discretes:D_SOD-323, F.Cu at (216.5, 89.0)
- added D1301: PMEG3010AESB, BR_Discretes:D_SOD-993-minimized, F.Cu at (258.1, 104.0)
- added D401: RB520S-30, BR_Discretes:D_SOD-523, F.Cu at (239.7, 69.6)
- added D402: RB520S-30, BR_Discretes:D_SOD-523, F.Cu at (239.7, 71.9)
- added D403: RB520S-30, BR_Discretes:D_SOD-523, F.Cu at (239.7, 74.3)
- added D404: RB520S-30, BR_Discretes:D_SOD-523, F.Cu at (239.7, 76.6)
- added J1001: TX_OUT_GAIN, BR_Connectors:PinHeader_1x02_P2.54mm_Vertical, F.Cu at (239.2, 90.6)
- added J101: POWER, BR_Connectors:KF128-2.54-2P, F.Cu at (54.5, 139.5)
- added J102: DEBUG, BR_Connectors_FFC_FPC:TE_2328702-6_1x06-1MP_P0.5mm_Horizontal, F.Cu at (117.7, 142.5)
- added J103: PORT1, BR_Connectors:RJ45-TH_RC01812, F.Cu at (95.0, 132.2)
- added J104: FPGA, BR_Connectors:HDR-SMD_20P-P2.54-V-M-R2-C10-S7.5, B.Cu at (107.3, 109.7)
- added J106: SYNC, BR_Connectors_JST:SM02B-GHS-TB, F.Cu at (110.7, 142.0)
- added J107: SONAR+, BR_Connectors:PinHeader_1x02_P2.54mm_Vertical, F.Cu at (128.5, 132.9)
- added J108: SONAR+, BR_Connectors:PinHeader_1x02_P2.54mm_Vertical, F.Cu at (128.5, 136.5)
- added J109: SONAR-, BR_Connectors:PinHeader_1x02_P2.54mm_Vertical, F.Cu at (135.5, 132.9)
- added J110: SONAR-, BR_Connectors:PinHeader_1x02_P2.54mm_Vertical, F.Cu at (135.5, 136.5)
- added J112: MOTOR, BR_Connectors_JST:SM04B-GHS-TB, F.Cu at (66.5, 142.0)
- added J1201: RFBT, BR_Connectors:PinHeader_1x02_P2.54mm_Vertical, F.Cu at (205.0, 97.0)
- added J1202: RDAC, BR_Connectors:PinHeader_1x02_P2.54mm_Vertical, F.Cu at (209.6, 97.0)
- added J401: RX_IN, BR_Connectors:PinHeader_1x02_P2.54mm_Vertical, F.Cu at (231.7, 53.9)
- added J402: PREAMP, BR_Connectors:PinHeader_2x03_P2.54mm_Vertical_SMD, F.Cu at (235.8, 63.6)
- added J403: BIAS_RES, BR_Connectors:PinHeader_1x02_P2.54mm_Vertical, F.Cu at (236.3, 53.9)
- added J404: BIAS_RES, BR_Connectors:PinHeader_1x02_P2.54mm_Vertical, F.Cu at (240.9, 53.9)
- added J405: GAIN_RES, BR_Connectors:PinHeader_1x02_P2.54mm_Vertical, F.Cu at (245.5, 53.9)
- added J406: LPF_CAP, BR_Connectors:PinHeader_1x02_P2.54mm_Vertical, F.Cu at (250.1, 53.9)
- added J407: VARAMP_OUT, BR_Connectors:PinHeader_1x02_P2.54mm_Vertical, F.Cu at (254.7, 53.9)
- added J501: LABEL, BR_Connectors:HDR-SMD_20P-P2.54-V-M-R2-C10-S7.5, F.Cu at (242.8, 26.1)
- added J502: LABEL, BR_Connectors:HDR-SMD_20P-P2.54-V-M-R2-C10-S7.5, F.Cu at (242.8, 35.6)
- added J601: CAP, BR_Connectors:PinHeader_1x02_P2.54mm_Vertical, F.Cu at (267.3, 23.6)
- added J901: OCTOSPI, BR_Connectors:PinHeader_2x06_P2.54mm_Vertical_SMD, B.Cu at (95.2, 88.5)
- added L1101: 2u2 2.2A, BR_Inductors:L_Taiyo-Yuden_NR-4018, F.Cu at (274.4, 24.0)
- added L1201: 10uH 30A, BR_Inductors:FC-SE2918-100M-28A, F.Cu at (195.7, 76.0)
- added L1301: 4u7 1.6A, BR_Inductors:L_1008_2520Metric, F.Cu at (254.5, 101.0)
- added L801: 10uH 10A, BR_Inductors:XR1265-100M, F.Cu at (32.5, 218.0)
- added NT1101: NetTie-2_0.18mm, BR_Virtual_Parts:NetTie-2_SMD_Pad_0.18mm_wide_long, F.Cu at (276.9, 29.1)
- added NT1201: Net_Tie_0201, BR_Virtual_Parts:Net_Tie_0201_1608Metric, F.Cu at (215.5, 93.1)
- added NT1501: NetTie-2_0.18mm, BR_Virtual_Parts:NetTie-2_SMD_Pad_0.18mm_wide_long, F.Cu at (270.2, 91.2)
- added NT801: NetTie-2_0.18mm, BR_Virtual_Parts:NetTie-2_SMD_Pad_0.18mm_wide_long, F.Cu at (41.0, 222.1)
- added Q1201: SQJ974EP, BR_SOP:PowerPAK_SO-8_Dual, F.Cu at (207.1, 105.2)
- added Q1501: DMN2990UDJ, BR_SOT:SOT-963, F.Cu at (268.1, 92.0)
- added R1001: 1M, BR_Passives:R_0201_0603Metric-minimized, F.Cu at (241.9, 85.3)
- added R1002: 1M, BR_Passives:R_0201_0603Metric-minimized, F.Cu at (241.9, 86.8)
- added R1003: 10k, BR_Passives:R_0201_0603Metric-minimized, F.Cu at (244.1, 80.6)
- added R1004: 1M, BR_Passives:R_0201_0603Metric-minimized, F.Cu at (244.1, 82.2)
- added R1005: 1M, BR_Passives:R_0201_0603Metric-minimized, F.Cu at (244.1, 83.7)
- added R1006: 10k, BR_Passives:R_0201_0603Metric-minimized, F.Cu at (244.1, 85.3)
- added R1007: 100k, BR_Passives:R_0201_0603Metric-minimized, F.Cu at (244.1, 86.8)
- added R1008: 100k, BR_Passives:R_0201_0603Metric-minimized, F.Cu at (246.3, 80.6)
- added R1009: 100k, BR_Passives:R_0201_0603Metric-minimized, F.Cu at (246.3, 82.2)
- added R101: 1k, BR_Passives:C_0402_1005Metric-minimized, F.Cu at (215.9, 22.2)
- added R1010: 100k, BR_Passives:R_0201_0603Metric-minimized, F.Cu at (246.3, 83.7)
- added R1011: 200R, BR_Passives:C_0402_1005Metric-minimized, F.Cu at (230.7, 88.1)
- added R1012: 50k, BR_Passives:RES-ADJ-SMD_3P-L3.8-W3.7_VGF39NCHXT, F.Cu at (244.4, 90.4)
- added R1013: 1k, BR_Passives:C_1210_3225Metric-minimized, F.Cu at (234.5, 90.2)
- added R1014: 1k, BR_Passives:C_1210_3225Metric-minimized, F.Cu at (234.5, 94.1)
- added R1015: 10mR, BR_Passives:R_0805_2012Metric, F.Cu at (239.1, 96.9)
- added R102: 1k, BR_Passives:C_0402_1005Metric-minimized, F.Cu at (215.9, 24.0)
- added R105: 100k, BR_Passives:C_0402_1005Metric-minimized, F.Cu at (215.9, 25.9)
- added R106: 100k, BR_Passives:C_0402_1005Metric-minimized, F.Cu at (215.9, 27.7)
- added R107: 100k, BR_Passives:C_0402_1005Metric-minimized, F.Cu at (215.9, 29.5)
- added R108: 100k, BR_Passives:C_0402_1005Metric-minimized, F.Cu at (218.5, 22.2)
- added R109: 100k, BR_Passives:C_0402_1005Metric-minimized, F.Cu at (218.5, 24.0)
- added R110: 100k, BR_Passives:C_0402_1005Metric-minimized, F.Cu at (218.5, 25.9)
- added R1101: 45k3, BR_Passives:C_0402_1005Metric-minimized, F.Cu at (278.4, 25.9)
- added R1102: 10k, BR_Passives:R_0201_0603Metric-minimized, F.Cu at (277.3, 27.6)
- added R111: 10k, BR_Passives:R_0201_0603Metric-minimized, F.Cu at (204.8, 58.8)
- added R1201: 1k, BR_Passives:R_0201_0603Metric-minimized, F.Cu at (219.9, 86.2)
- added R1202: 68k1, BR_Passives:C_0402_1005Metric-minimized, F.Cu at (218.4, 67.7)
- added R1203: 2k2, BR_Passives:R_0402_1005Metric-minimized, F.Cu at (218.4, 69.6)
- added R1204: 75k, BR_Passives:R_0402_1005Metric-minimized, F.Cu at (218.4, 71.4)
- added R1205: 3mR, BR_Passives:R_2512_6332Metric, F.Cu at (216.2, 105.3)
- added R1206: 137k, BR_Passives:C_0402_1005Metric-minimized, F.Cu at (221.0, 65.9)
- added R1207: 10k, BR_Passives:C_0402_1005Metric-minimized, F.Cu at (221.0, 67.7)
- added R1208: 24k9, BR_Passives:C_0402_1005Metric-minimized, F.Cu at (221.0, 69.6)
- added R1301: 51k, BR_Passives:C_0402_1005Metric-minimized, F.Cu at (250.7, 103.8)
- added R1302: 13.3k, BR_Passives:C_0402_1005Metric-minimized, F.Cu at (250.7, 105.6)
- added R1303: 62k, BR_Passives:C_0402_1005Metric-minimized, F.Cu at (250.7, 107.4)
- added R1501: 100k, BR_Passives:C_0402_1005Metric-minimized, F.Cu at (275.2, 88.1)
- added R1502: 2R2, BR_Passives:R_0402_1005Metric-minimized, F.Cu at (277.8, 80.8)
- added R1503: 2R2, BR_Passives:R_0402_1005Metric-minimized, F.Cu at (277.8, 82.6)
- added R1504: 2R2, BR_Passives:R_0402_1005Metric-minimized, F.Cu at (277.8, 84.5)
- added R1505: 2R2, BR_Passives:R_0402_1005Metric-minimized, F.Cu at (277.8, 86.3)
- added R1506: 100k, BR_Passives:C_0402_1005Metric-minimized, F.Cu at (277.8, 88.1)
- added R1601: 0R, BR_Passives:R_0603_1608Metric, F.Cu at (275.5, 43.3)
- added R1602: 0R, BR_Passives:R_0603_1608Metric, F.Cu at (275.5, 45.8)
- added R1603: 330k, BR_Passives:C_0402_1005Metric-minimized, F.Cu at (272.2, 46.3)
- added R1604: 10k, BR_Passives:C_0402_1005Metric-minimized, F.Cu at (272.2, 48.1)
- added R304: 10k, BR_Passives:C_0402_1005Metric-minimized, F.Cu at (267.6, 38.9)
- added R305: 10k, BR_Passives:C_0402_1005Metric-minimized, F.Cu at (267.6, 40.7)
- added R401: 100R, BR_Passives:C_0201_0603Metric-minimized, F.Cu at (248.6, 74.0)
- added R402: 100R, BR_Passives:C_0201_0603Metric-minimized, F.Cu at (248.6, 75.5)
- added R403: 100R, BR_Passives:C_0201_0603Metric-minimized, F.Cu at (248.6, 77.1)
- added R404: 470R, BR_Passives:C_0402_1005Metric-minimized, F.Cu at (246.1, 61.5)
- added R405: 470R, BR_Passives:C_0402_1005Metric-minimized, F.Cu at (246.1, 63.4)
- added R406: 75R, BR_Passives:C_0402_1005Metric-minimized, F.Cu at (246.1, 65.2)
- added R407: 75R, BR_Passives:C_0402_1005Metric-minimized, F.Cu at (246.1, 67.1)
- added R408: 0R, BR_Passives:R_0603_1608Metric, F.Cu at (231.4, 76.3)
- added R409: 1k, BR_Passives:C_0402_1005Metric-minimized, F.Cu at (246.1, 68.9)
- added R410: 1k, BR_Passives:C_0402_1005Metric-minimized, F.Cu at (246.1, 70.7)
- added R411: 1k, BR_Passives:C_0402_1005Metric-minimized, F.Cu at (248.7, 59.7)
- added R412: 1k, BR_Passives:C_0402_1005Metric-minimized, F.Cu at (248.7, 61.5)
- added R413: 2k, BR_Passives:C_0402_1005Metric-minimized, F.Cu at (248.7, 63.4)
- added R414: 2k, BR_Passives:C_0402_1005Metric-minimized, F.Cu at (248.7, 65.2)
- added R501: 20k, BR_Passives:R_0201_0603Metric-minimized, F.Cu at (232.8, 43.1)
- added R502: 2k, BR_Passives:C_0402_1005Metric-minimized, F.Cu at (233.0, 41.4)
- added R601: 100k, BR_Passives:C_0402_1005Metric-minimized, F.Cu at (259.4, 33.2)
- added R701: 2k49, BR_Passives:C_0402_1005Metric-minimized, F.Cu at (272.9, 98.3)
- added R702: 2k49, BR_Passives:C_0402_1005Metric-minimized, F.Cu at (272.9, 100.2)
- added R703: 75R, BR_Passives:C_0402_1005Metric-minimized, F.Cu at (272.9, 102.0)
- added R704: 75R, BR_Passives:C_0402_1005Metric-minimized, F.Cu at (275.5, 96.5)
- added R705: 6k49, BR_Passives:C_0402_1005Metric-minimized, F.Cu at (275.5, 98.3)
- added R706: 30k, BR_Passives:C_0402_1005Metric-minimized, F.Cu at (275.5, 100.2)
- added R707: 1M, BR_Passives:C_0402_1005Metric-minimized, F.Cu at (275.5, 102.0)
- added R708: 2k49, BR_Passives:C_0402_1005Metric-minimized, F.Cu at (278.1, 96.5)
- added R709: 2k49, BR_Passives:C_0402_1005Metric-minimized, F.Cu at (278.1, 98.3)
- added R710: 2k49, BR_Passives:C_0402_1005Metric-minimized, F.Cu at (278.1, 100.2)
- added R711: 2k49, BR_Passives:C_0402_1005Metric-minimized, F.Cu at (278.1, 102.0)
- added R801: 20k, BR_Passives:C_0402_1005Metric-minimized, F.Cu at (26.0, 231.5)
- added R802: 10k, BR_Passives:C_0402_1005Metric-minimized, F.Cu at (26.0, 233.4)
- added R803: 100k, BR_Passives:C_0402_1005Metric-minimized, F.Cu at (28.6, 226.0)
- added R804: 51k, BR_Passives:C_0402_1005Metric-minimized, F.Cu at (28.6, 227.9)
- added R805: 2R2, BR_Passives:R_0402_1005Metric-minimized, F.Cu at (28.6, 229.7)
- added R806: 2R2, BR_Passives:R_0402_1005Metric-minimized, F.Cu at (28.6, 231.5)
- added R807: 2k2, BR_Passives:R_0402_1005Metric-minimized, F.Cu at (28.6, 233.4)
- added R808: 24k9, BR_Passives:C_0402_1005Metric-minimized, F.Cu at (31.2, 226.0)
- added R809: 4k99, BR_Passives:C_0402_1005Metric-minimized, F.Cu at (31.2, 227.9)
- added R810: 681R, BR_Passives:C_0402_1005Metric-minimized, F.Cu at (31.2, 229.7)
- added T101: B65655B0010X000, BR_Inductors:B65655B0010X000, F.Cu at (138.4, 118.5)
- added TH101: 10k 3380K, BR_Passives:R_0201_0603Metric-minimized, F.Cu at (204.8, 61.9)
- added TP1001: POT2, BR_Virtual_Parts:TP_SQUARE_TH_1mm, F.Cu at (230.6, 90.2)
- added TP1002: POT1, BR_Virtual_Parts:TP_SQUARE_TH_1mm, F.Cu at (230.5, 92.0)
- added TP302: TP_ROUND_TH_300um, BR_Virtual_Parts:TP_ROUND_SMT_300um, F.Cu at (258.8, 36.9)
- added TP303: TP_ROUND_TH_300um, BR_Virtual_Parts:TP_ROUND_SMT_300um, F.Cu at (258.8, 38.4)
- added TP304: TP_ROUND_TH_300um, BR_Virtual_Parts:TP_ROUND_SMT_300um, F.Cu at (258.8, 39.9)
- added TP305: TP_ROUND_TH_300um, BR_Virtual_Parts:TP_ROUND_SMT_300um, F.Cu at (258.8, 41.4)
- added TP306: TP_ROUND_TH_300um, BR_Virtual_Parts:TP_ROUND_SMT_300um, F.Cu at (258.8, 42.9)
- added TP307: TP_ROUND_TH_300um, BR_Virtual_Parts:TP_ROUND_SMT_300um, F.Cu at (258.8, 44.4)
- added TP308: TP_ROUND_TH_300um, BR_Virtual_Parts:TP_ROUND_SMT_300um, F.Cu at (258.8, 45.9)
- added TP310: TP_ROUND_TH_300um, BR_Virtual_Parts:TP_ROUND_SMT_300um, F.Cu at (260.3, 36.9)
- added TP311: TP_ROUND_TH_300um, BR_Virtual_Parts:TP_ROUND_SMT_300um, F.Cu at (260.3, 38.4)
- added TP312: TP_ROUND_TH_300um, BR_Virtual_Parts:TP_ROUND_SMT_300um, F.Cu at (260.3, 39.9)
- added TP313: TP_ROUND_TH_300um, BR_Virtual_Parts:TP_ROUND_SMT_300um, F.Cu at (260.3, 41.4)
- added TP317: TP_ROUND_TH_300um, BR_Virtual_Parts:TP_ROUND_SMT_300um, F.Cu at (260.3, 42.9)
- added TP318: TP_ROUND_TH_300um, BR_Virtual_Parts:TP_ROUND_SMT_300um, F.Cu at (260.3, 44.4)
- added TP319: TP_ROUND_TH_300um, BR_Virtual_Parts:TP_ROUND_SMT_300um, F.Cu at (260.3, 45.9)
- added TP320: TP_ROUND_TH_300um, BR_Virtual_Parts:TP_ROUND_SMT_300um, F.Cu at (261.8, 36.9)
- added TP327: TP_ROUND_TH_300um, BR_Virtual_Parts:TP_ROUND_SMT_300um, F.Cu at (261.8, 38.4)
- added TP331: TP_ROUND_TH_300um, BR_Virtual_Parts:TP_ROUND_SMT_300um, F.Cu at (261.8, 39.9)
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- renumbered C61 to C105, C7 to C201, C11 to C302, C31 to C303, C50 to C304, C10 to C306, C12 to C307, C28 to C309, C30 to C311, C54 to C312, C45 to C313, C32 to C314, C33 to C315, C34 to C317, C35 to C318, C36 to C319, C38 to C320, C39 to C321, C40 to C322, C41 to C323, C42 to C324, C43 to C325, D2 to D101, D1 to D301, H1 to H101, H2 to H102, H3 to H103, H4 to H104, Q1 to Q101, R36 to R103, R15 to R201, R18 to R202, R32 to R301, R31 to R302, R35 to R303, T1 to T701, TP30 to TP301, TP49 to TP309, TP3 to TP314, TP39 to TP315, TP4 to TP316, TP48 to TP321, TP47 to TP322, TP46 to TP323, TP45 to TP324, TP22 to TP325, TP37 to TP326, TP9 to TP328, TP10 to TP329, TP12 to TP330, TP14 to TP332, TP15 to TP334, TP17 to TP335, TP18 to TP336, TP7 to TP337, TP8 to TP338, TP35 to TP339, TP36 to TP340, TP23 to TP343, TP24 to TP344, TP25 to TP345, TP26 to TP346, TP13 to TP347, TP27 to TP348, TP28 to TP349, TP29 to TP350, TP16 to TP351, TP40 to TP359, TP41 to TP360, TP42 to TP361, TP43 to TP362, TP44 to TP363, TP50 to TP364, TP11 to TP365, U6 to U301, U1 to U701, X1 to X301
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Connections:
- net /MCU/DAC renamed /TX_SIG
- net /MCU/I2C4.SCL renamed /I2C4.SCL
- net /MCU/I2C4.SDA renamed /I2C4.SDA
- net /MCU/ISENSE renamed /TX_I_SENSE
- net /MCU/SWCLK renamed /SWCLK
- net /MCU/SWDIO renamed /SWDIO
- net /MCU/USART1.RX renamed /USART1.RX
- net /MCU/USART1.TX renamed /USART1.TX
- net /MCU/nRST renamed /nRST
- C201 pad 1: /Power/V_SENSE -> /V_SENSE
- C301 pad 1: 5V -> 3V3
- C301 pad 2: /3V3 Buck/PGND -> GND
- C901 pad 1: 5V -> 3V3
- C901 pad 2: /1V1 Buck/PGND -> GND
- C902 pad 1: 1V1 -> 3V3
- C902 pad 2: /1V1 Buck/PGND -> GND
- H101 pad 1: unconnected-(H1-Pad1) -> Net-(C101-Pad1)
- H102 pad 1: unconnected-(H2-Pad1) -> Net-(C103-Pad1)
- H103 pad 1: unconnected-(H3-Pad1) -> Net-(C107-Pad1)
- H104 pad 1: unconnected-(H4-Pad1) -> Net-(C109-Pad1)
- J111 pad 1: /SONAR_SIGNAL -> /SONAR+
- J111 pad 2: GND -> /SONAR-
- L301 pad 1: /3V3 Buck/SW -> Net-(C308-Pad1)
- L301 pad 2: 3V3 -> Net-(U301-VLXSMPS)
- R104 pad 2: /3V3 Buck/RSET -> /VTHERM
- R112 pad 1: 1V1 -> 3V3
- R112 pad 2: /1V1 Buck/RSET -> /I2C1.SCL
- R201 pad 1: /Power/VIN_PROTECTED -> /V_SENSE
- R201 pad 2: /Power/V_SENSE -> VIN_PROTECTED
- R202 pad 1: /Power/V_SENSE -> /V_SENSE
- T701 pad 1: /Ethernet/ETH.TX+ -> /Ethernet/TD_P
- T701 pad 10: unconnected-(T1-Pad10) -> Net-(R704-Pad2)
- T701 pad 11: Net-(U1-RD_P) -> /ETH.RX+
- T701 pad 14: Net-(U1-TD_N) -> /ETH.TX-
- T701 pad 15: unconnected-(T1-Pad15) -> Net-(R703-Pad2)
- T701 pad 16: Net-(U1-TD_P) -> /ETH.TX+
- T701 pad 2: unconnected-(T1-Pad2) -> Net-(C708-Pad1)
- T701 pad 3: /Ethernet/ETH.TX- -> /Ethernet/TD_N
- T701 pad 6: /Ethernet/ETH.RX+ -> /Ethernet/RD_P
- T701 pad 7: unconnected-(T1-Pad7) -> Net-(C708-Pad1)
- T701 pad 8: /Ethernet/ETH.RX- -> /Ethernet/RD_N
- T701 pad 9: Net-(U1-RD_N) -> /ETH.RX-
- TP309 pad 1: /MCU/OCTOSPI1.IO4 -> /OCTOSPI1.IO4
- TP314 pad 1: /MCU/PHY_nRST -> /PHY_nRST
- TP321 pad 1: /MCU/OCTOSPI1.IO3 -> /OCTOSPI1.IO3
- TP322 pad 1: /MCU/OCTOSPI1.IO0 -> /OCTOSPI1.IO0
- TP323 pad 1: /MCU/OCTOSPI1.IO1 -> /OCTOSPI1.IO1
- TP324 pad 1: /MCU/OCTOSPI1.CLK -> /OCTOSPI1.CLK
- TP325 pad 1: /MCU/VTHERM -> /VTHERM
- TP326 pad 1: /MCU/VSENSE -> /V_SENSE
- TP330 pad 1: /MCU/MAC.MDIO -> /MAC.MDIO
- TP334 pad 1: /MCU/MAC.RXDV -> /MAC.CRSDV
- TP339 pad 1: /MCU/OCTOSPI1.DQS -> /OCTOSPI1.DQS
- TP340 pad 1: /MCU/OCTOSPI1.NCLK -> /OCTOSPI1.NCLK
- TP343 pad 1: /MCU/MAC.RXER -> /MAC.RXER
- TP344 pad 1: /MCU/MAC.TXEN -> /MAC.TXEN
- TP345 pad 1: /MCU/MAC.TXD0 -> /MAC.TXD0
- TP346 pad 1: /MCU/MAC.TXD1 -> /MAC.TXD1
- TP348 pad 1: /MCU/MAC.MDC -> /MAC.MDC
- TP349 pad 1: /MCU/MAC.RXD0 -> /MAC.RXD0
- TP350 pad 1: /MCU/MAC.RXD1 -> /MAC.RXD1
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Routing:
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- removed copper zone on F.Cu, net /1V1 Buck/PGND
- removed copper zone on F.Cu, net /3V3 Buck/PGND
- removed copper zone on F.Cu, net 1V1
- removed copper zone on F.Cu, net 3V3
- removed copper zone on F.Cu, net 5V
Other:
- copper layers 2 -> 6

Commit message: minor schematic updates + subcircuit layout
Parts:
- added C1607: 2u2F 10V, BR_Passives:C_0402_1005Metric-minimized, F.Cu at (62.9, 138.8)
- C809, L801, R1601, R1602: moved to B.Cu
- U402: footprint Package_SO:SOIC-8-1EP_3.9x4.9mm_P1.27mm_EP2.41x3.3mm -> BR_SO:SOIC-8_3.9x4.9mm_P1.27mm
- moved U1601 232.6 mm to (64.6, 135.2), turned to 90 degrees
- moved R1601 230.8 mm to (63.1, 133.6)
- moved C1603 230.8 mm to (62.9, 138.0), turned to 180 degrees
- moved C1604 230.7 mm to (61.7, 137.1), turned to 90 degrees
- moved C1605 230.4 mm to (61.7, 135.4), turned to 90 degrees
- moved R1602 227.0 mm to (66.1, 133.6), turned to 180 degrees
- moved C1601 227.0 mm to (68.1, 136.4), turned to -90 degrees
- moved C1602 226.9 mm to (67.3, 136.4), turned to -90 degrees
- moved R1603 223.7 mm to (65.7, 132.4)
- moved C1606 223.7 mm to (67.7, 135.1)
- moved R1604 221.9 mm to (67.7, 134.3), turned to 180 degrees
- moved C108 198.0 mm to (44.7, 133.6), turned to 180 degrees
- moved C110 196.3 mm to (44.7, 131.9), turned to 180 degrees
- moved C114 186.1 mm to (74.7, 153.8), turned to 90 degrees
- moved C102 184.4 mm to (44.6, 129.9), turned to 180 degrees
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Connections:
- net Net-(C809-Pad2) renamed /Power/5V Buck/SW
- J112 pad 3: /MOTOR_B+ -> /MOTOR_B-
- J112 pad 4: /MOTOR_B- -> /MOTOR_B+
- U1601 pad 25: (no net) -> GND
Routing:
- net GND: vias 14 -> 17
- net 3V3: vias 14 -> 17
- net /PSRAM_nRST: vias 1 -> 2
- net /OCTOSPI1.NCS: vias 1 -> 2
- net /OCTOSPI1.NCLK: vias 1 -> 2
- net /OCTOSPI1.IO7: vias 1 -> 2
- net /OCTOSPI1.IO6: vias 1 -> 2
- net /OCTOSPI1.IO5: vias 1 -> 2
- net /OCTOSPI1.IO4: vias 1 -> 2
- net /OCTOSPI1.IO3: vias 1 -> 2
- net /OCTOSPI1.IO2: vias 1 -> 2
- net /OCTOSPI1.IO1: vias 1 -> 2
- net /OCTOSPI1.IO0: vias 1 -> 2
- net /OCTOSPI1.DQS: vias 1 -> 2
- net /OCTOSPI1.CLK: vias 1 -> 2

Commit message: Start 5V buck layout
Parts:
- C809: moved to F.Cu
- moved C1401 282.5 mm to (453.8, -65.4)
- moved C1402 282.5 mm to (456.2, -65.5)
- moved U1401 282.5 mm to (454.9, -68.5)
- moved R807 237.8 mm to (96.6, -75.9)
- moved C810 232.5 mm to (98.5, -70.8), turned to 180 degrees
- moved C808 231.8 mm to (98.1, -72.0), turned to -90 degrees
- moved R806 230.1 mm to (101.1, -66.1)
- moved R808 219.8 mm to (93.5, -65.8)
- moved R805 219.3 mm to (77.8, -68.7)
- moved C1201 215.8 mm to (197.6, -85.1)
- moved C1202 215.8 mm to (198.9, -76.7)
- moved C1203 215.8 mm to (197.6, -83.3)
- moved C1204 215.8 mm to (201.8, -66.3)
- moved C1205 215.8 mm to (197.8, -59.6)
- moved C1206 215.8 mm to (197.6, -81.4)
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Routing:
- added copper zone on F.Cu, net /Power/5V Buck/PGND
Other:
- board size 110 x 60 mm -> 540 x 106.9 mm

Commit message: Lay out 5V buck converter
Parts:
- added Q1502: MMBT3904L, BR_SOT:SOT-23, F.Cu at (373.0, 57.4)
- added Q1503: MMBT3904L, BR_SOT:SOT-23, F.Cu at (373.0, 61.7)
- added R1507: 5k1, BR_Passives:C_0402_1005Metric-minimized, F.Cu at (376.6, 55.4)
- added R1508: 24k9, BR_Passives:C_0402_1005Metric-minimized, F.Cu at (376.6, 57.2)
- L801: moved to F.Cu
- Q1501: value DMN2990UDJ -> MMBT3904L; footprint BR_SOT:SOT-963 -> BR_SOT:SOT-23
- R1501: value 100k -> 24k9
- R1506: value 100k -> 5k1
- moved Q1501 111.9 mm to (373.0, 53.0)
- moved R1501 107.7 mm to (376.6, 51.7)
- moved R1506 104.7 mm to (376.6, 53.6)
- moved U1201 46.3 mm to (196.3, -98.5)
- moved C1202 43.0 mm to (159.2, -60.0)
- moved NT801 38.4 mm to (78.3, -75.8), turned to 180 degrees
- moved R809 24.1 mm to (100.6, -68.0), turned to 90 degrees
- moved C811 22.6 mm to (99.7, -67.9), turned to 90 degrees
- moved R805 20.9 mm to (98.1, -73.8), turned to 90 degrees
- moved R803 20.1 mm to (97.7, -67.6), turned to 0 degrees
- moved R801 20.0 mm to (96.6, -66.9), turned to 180 degrees
- moved R804 19.4 mm to (98.1, -68.8), turned to 90 degrees
- moved R810 19.1 mm to (98.1, -71.0), turned to 90 degrees
- moved C807 16.5 mm to (99.9, -73.8), turned to 0 degrees
- moved C812 15.1 mm to (92.0, -66.0), turned to 90 degrees
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Connections:
- C1501 pad 1: /TX/Digital Drive/5V -> 5V
- C1506 pad 1: /TX/Digital Drive/5V -> 5V
- Q1501 pad 1: Net-(U1501-SD) -> Net-(Q1501-B)
- Q1501 pad 3: /TX/Digital Drive/5V -> Net-(Q1501-C)
- R1501 pad 1: /SD0 -> /TX/Digital Drive/3V3
- R1501 pad 2: GND -> Net-(Q1501-B)
- R1502 pad 1: /TX/Digital Drive/5V -> 5V
- R1504 pad 2: /TX/Digital Drive/5V -> 5V
- R1506 pad 1: /SD1 -> 5V
- R1506 pad 2: GND -> Net-(Q1501-C)
- U1501 pad 3: Net-(U1501-SD) -> /SD0
- U1501 pad 5: /TX/Digital Drive/5V -> 5V
- U1502 pad 3: Net-(U1502-SD) -> /SD1
- U1502 pad 5: /TX/Digital Drive/5V -> 5V
Routing:
- net /Power/5V Buck/SW: track 0.00 -> 18.1 mm, vias 0 -> 3
- net VIN_PROTECTED: track 0.00 -> 12.7 mm, vias 0 -> 3
- net Net-(U801-PVDD): track 0.00 -> 8.66 mm, vias 0 -> 2
- net Net-(U801-FB): track 0.00 -> 5.39 mm
- net GND: track 0.00 -> 4.73 mm, vias 17 -> 22
- net Net-(U801-VDD): track 0.00 -> 2.68 mm
- net Net-(U801-EN): track 0.00 -> 2.65 mm
- net Net-(U801-FREQ): track 0.00 -> 2.42 mm
- net Net-(U801-SVIN): track 0.00 -> 2.30 mm
- net 5V: track 0.00 -> 2.24 mm, vias 0 -> 29
- net Net-(U801-ILIM): track 0.00 -> 1.80 mm
- net Net-(U801-BST): track 0.00 -> 1.33 mm
- net /Power/5V Buck/PGND: track 0.00 -> 1.23 mm
- net Net-(C810-Pad1): track 0.00 -> 0.85 mm
- added copper zone on F.Cu, net /Power/5V Buck/SW
- added copper zone on F.Cu, net 5V
- added copper zone on B.Cu, net GND
- added copper zone on F.Cu, net GND
- added copper zone on In1.Cu, net GND
- added copper zone on In2.Cu, net GND
- added copper zone on In3.Cu, net GND
- added copper zone on In4.Cu, net GND
- added copper zone on F.Cu, net VIN_PROTECTED
Other:
- board text added: "${REFERENCE}"

Commit message: Lay out 3V3 buck, 7V boost, and 5V LDO
Parts:
- moved C1202 59.2 mm to (218.4, -61.9), turned to 90 degrees
- moved L1201 50.6 mm to (212.4, -38.4), turned to 180 degrees
- moved U1201 38.8 mm to (213.4, -63.7), turned to 90 degrees
- moved C1209 35.9 mm to (237.9, -59.8)
- moved C1210 35.9 mm to (237.9, -57.6)
- moved C1208 25.6 mm to (197.6, -62.9), turned to 90 degrees
- moved C1303 22.9 mm to (389.3, -58.7)
- moved R1302 22.5 mm to (390.9, -58.7)
- moved Q1201 22.5 mm to (207.2, -59.1), turned to -90 degrees
- moved R1301 21.4 mm to (390.7, -63.4)
- moved C1301 21.3 mm to (389.1, -63.4)
- moved R1303 21.1 mm to (389.4, -57.0), turned to 180 degrees
- moved C1205 19.9 mm to (178.3, -63.8)
- moved C1204 19.9 mm to (182.3, -70.5)
- moved NT1201 19.9 mm to (177.9, -62.0)
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Routing:
- net 5V: track 2.24 -> 11.3 mm, vias 29 -> 36
- net GND: track 4.73 -> 8.26 mm, vias 22 -> 25
- net Net-(U1301-FB): track 0.00 -> 3.28 mm
- net Net-(U1101-FB): track 0.00 -> 2.93 mm
- net 3V3: track 0.00 -> 2.68 mm, vias 17 -> 20
- net Net-(U1301-EN): track 0.00 -> 1.41 mm
- net /Power/7V: track 0.00 -> 1.29 mm, vias 0 -> 3
- net RX_5V: track 0.00 -> 1.13 mm, vias 0 -> 1
- added copper zone on F.Cu, net /Power/3V3 Buck/PGND
- added copper zone on F.Cu, net /Power/3V3 Buck/SW
- added copper zone on F.Cu, net /Power/7V
- added copper zone on F.Cu, net Net-(D1301-A)
