File: 5v_buck.kicad_sch (KiCad schematic)
At the start: 24 parts, among them U801 MIC28517T-E/PHA

Commit message: adding test pads + minor schematic edits
Parts:
- added D801: LABEL, BR_Optoelectronics:LED_0603_1608Metric, symbol BR_Optoelectronic:LTST-C191KGKT
- added R811: 330R, BR_Passives:C_0402_1005Metric-minimized, symbol BR_Resistors_0402:R_0402_330R
- added TP801: 5V, BR_Connectors:TEST-TH_BD2.54-P1.4_RED, symbol BR_Connectors:TP_Ring_PTH
Connections:
- net GND: now also D801.1 (K)
- net VOUT: now also R811.1, TP801.1
- new net: D801.2 (A), R811.2

Commit message: preboard review of updates
Parts:
- R811: value 330R -> 3k; symbol BR_Resistors_0402:R_0402_330R -> BR_Resistors_0402:R_0402_3k; BRE Number BRE-000331 -> BRE-000337; JLCPCB Part Num C105875 -> C137987; Manufacturer Part Num RC0402FR-07330RL -> RC0402FR-073KL; Supplier 2 Mouser -> DigiKey; Supplier Part Num 1 311-330LRCT-ND -> 311-3KLRCT-ND; Supplier Part Num 2 603-RC0402FR-07330RL -> 311-3KLRTR-ND; Supplier Part Num 3 C105875 -> C137987
Changed lines of the file:
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@@
 	)
 	(symbol
-		(lib_id "BR_Resistors_0402:R_0402_330R")
+		(lib_id "BR_Resistors_0402:R_0402_3k")
 		(at 190.5 129.54 0)
 		(unit 1)
@@
 			)
 		)
-		(property "Value" "330R"
+		(property "Value" "3k"
 			(at 193.04 130.8099 0)
 			(effects
@@
 			)
 		)
-		(property "Datasheet" "https://www.yageo.com/upload/media/product/products/datasheet/rchip/PYu-RC_Group_51_RoHS_L_12.pdf"
+		(property "Datasheet" "https://www.yageo.com/upload/media/product/app/datasheet/rchip/pyu-rc_group_51_rohs_l.pdf"
 			(at 190.5 55.88 0)
 			(effects
@@
 			)
 		)
-		(property "Description" "330R 1% 100ppm 62.5mW Thick Film Resistor 0402"
+		(property "Description" "3k 1% 100ppm 62.5mW Thick Film Resistor 0402"
 			(at 190.5 66.04 0)
 			(effects
@@
 			)
 		)
-		(property "Manufacturer Part Num" "RC0402FR-07330RL"
+		(property "Manufacturer Part Num" "RC0402FR-073KL"
 			(at 190.5 60.96 0)
 			(effects
@@
 			)
 		)
-		(property "BRE Number" "BRE-000331"
+		(property "BRE Number" "BRE-000337"
 			(at 190.5 63.5 0)
 			(effects
@@
 			)
 		)
-		(property "Supplier Part Num 1" "311-330LRCT-ND"
+		(property "Supplier Part Num 1" "311-3KLRCT-ND"
 			(at 190.5 71.12 0)
 			(effects
@@
 			)
 		)
-		(property "Supplier 2" "Mouser"
+		(property "Supplier 2" "DigiKey"
 			(at 190.5 73.66 0)
 			(effects
@@
 			)
 		)
-		(property "Supplier Part Num 2" "603-RC0402FR-07330RL"
+		(property "Supplier Part Num 2" "311-3KLRTR-ND"
 			(at 190.5 76.2 0)
 			(effects
@@
 			)
 		)
-		(property "Supplier Part Num 3" "C105875"
+		(property "Supplier Part Num 3" "C137987"
 			(at 190.5 81.28 0)
 			(effects
@@
 			)
 		)
-		(property "JLCPCB Part Num" "C105875"
+		(property "JLCPCB Part Num" "C137987"
 			(at 190.5 83.82 0)
 			(effects

Commit message: various improvements
Parts:
- D801: value LABEL -> 5V
Changed lines of the file:
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@@
 			)
 		)
-		(property "Value" "LABEL"
+		(property "Value" "5V"
 			(at 194.31 141.0334 90)
 			(effects

Commit message: clarified silkscreen labels
Parts:
- U801: value MIC28517T-E/PHA -> BUCK CONVERTER
Changed lines of the file:
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@@
 			)
 		)
-		(property "Value" "MIC28517T-E/PHA"
+		(property "Value" "BUCK CONVERTER"
 			(at 144.78 52.07 0)
 			(effects

Commit message: last checks + board characteristics tables
Parts:
- added TP802: GND, BR_Connectors:TEST-TH_BD2.54-P1.4_RED, symbol BR_Connectors:TP_Ring_PTH
- C806: JLCPCB Part Num C20044523 -> C20044522
Connections:
- net GND: now also TP802.1
