File: stepper_driver.kicad_sch (KiCad schematic)
At the start: 12 parts, among them U1601 DRV8426RGER

Commit message: added net tie to stepper motor PGND + various routing
Parts:
- added NT1601: NetTie-2_0.18mm, BR_Virtual_Parts:NetTie-2_SMD_Pad_0.18mm_wide, symbol BR_Virtual_Parts:NetTie-2_0.18mm
Connections:
- net GND: now also NT1601.2
- net PGND: now also NT1601.1

Commit message: preboard review of updates
Connections:
- net GND: no longer U1601.25 (EP)
- net PGND: now also U1601.25 (EP)
Other:
- note removed: "EDIT FOOTPRINT OR SYMBOL PIN EP = 25"
Changed lines of the file:
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@@
 		)
 	)
-	(text "EDIT FOOTPRINT OR SYMBOL PIN EP = 25"
-		(exclude_from_sim no)
-		(at 182.372 131.064 0)
-		(effects
-			(font
-				(size 1.27 1.27)
-			)
-		)
-	)
 	(text "DECAY MODE SETTINGS: Smart Tune Ripple Control"
 		(exclude_from_sim no)
@@
 	)
 	(junction
-		(at 160.02 128.27)
-		(diameter 0)
-		(color 0 0 0 0)
-	)
-	(junction
 		(at 138.43 69.85)
 		(diameter 0)
@@
 	(wire
 		(pts
-			(xy 160.02 128.27) (xy 160.02 132.08)
-		)
-		(stroke
-			(width 0)
-			(type default)
-		)
-	)
-	(wire
-		(pts
-			(xy 160.02 128.27) (xy 163.83 128.27)
+			(xy 160.02 124.46) (xy 160.02 132.08)
 		)
 		(stroke
@@
 	(wire
 		(pts
-			(xy 123.19 76.2) (xy 142.24 76.2)
+			(xy 163.83 124.46) (xy 163.83 133.35)
 		)
 		(stroke
@@
 	(wire
 		(pts
-			(xy 151.13 144.78) (xy 151.13 151.13)
+			(xy 123.19 76.2) (xy 142.24 76.2)
 		)
 		(stroke
@@
 	(wire
 		(pts
-			(xy 106.68 86.36) (xy 142.24 86.36)
+			(xy 151.13 144.78) (xy 151.13 151.13)
 		)
 		(stroke
@@
 	(wire
 		(pts
-			(xy 167.64 144.78) (xy 163.83 144.78)
+			(xy 106.68 86.36) (xy 142.24 86.36)
 		)
 		(stroke
@@
 	(wire
 		(pts
-			(xy 160.02 124.46) (xy 160.02 128.27)
+			(xy 167.64 144.78) (xy 163.83 144.78)
 		)
 		(stroke
@@
 	(wire
 		(pts
-			(xy 163.83 128.27) (xy 163.83 124.46)
-		)
-		(stroke
-			(width 0)
-			(type default)
-		)
-	)
-	(wire
-		(pts
 			(xy 180.34 119.38) (xy 180.34 121.92)
 		)
@@
 		(effects
 			(font
+				(size 1.27 1.27)
+			)
+			(justify left bottom)
+		)
+	)
+	(label "PGND"
+		(at 163.83 133.35 90)
+		(effects
+			(font

Commit message: Rev A release files
Parts:
- C1606: JLCPCB Part Num C528974 -> C23692972
Changed lines of the file:
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@@
 			)
 		)
-		(property "JLCPCB Part Num" "C528974"
+		(property "JLCPCB Part Num" "C23692972"
 			(at 180.34 71.12 0)
 			(effects

Commit message: refactoring tx a bit
Parts:
- NT1601: value NetTie-2_0.18mm -> Net_Tie_0201; footprint BR_Virtual_Parts:NetTie-2_SMD_Pad_0.18mm_wide -> BR_Virtual_Parts:Net_Tie_0201_1608Metric; symbol BR_Virtual_Parts:NetTie-2_0.18mm -> BR_Virtual_Parts:Net_Tie_0201
Changed lines of the file:
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@@
 	)
 	(symbol
-		(lib_id "BR_Virtual_Parts:NetTie-2_0.18mm")
+		(lib_id "BR_Virtual_Parts:Net_Tie_0201")
 		(at 160.02 144.78 90)
 		(unit 1)
@@
 			)
 		)
-		(property "Value" "NetTie-2_0.18mm"
+		(property "Value" "Net_Tie_0201"
 			(at 160.02 142.24 90)
 			(effects
@@
 			)
 		)
-		(property "Footprint" "BR_Virtual_Parts:NetTie-2_SMD_Pad_0.18mm_wide"
+		(property "Footprint" "BR_Virtual_Parts:Net_Tie_0201_1608Metric"
 			(at 160.274 143.764 90)
 			(effects
