File: stepper_driver.kicad_sch (KiCad schematic)
At the start: 13 parts, among them U1601 DRV8426RGER

Commit message: more work
Parts:
- C1606: JLCPCB Part Num C23692972 -> C528974

Commit message: more work
Parts:
- renumbered C1607 to C1601, C1601 to C1602, C1602 to C1603, C1603 to C1604, C1604 to C1605, C1605 to C1606, C1606 to C1607
Changed lines of the file:
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@@
 		(in_pos_files no)
 		(dnp no)
-		(property "Reference" "#PWR01608"
+		(property "Reference" "#PWR01610"
 			(at 106.68 85.09 0)
 			(hide yes)
@@
 			(project "PingDevKit"
 				(path "/2a5ce3ef-537a-4122-a1be-ef76186bc0d7/a659e729-f286-4529-89a9-b647d33044af"
-					(reference "#PWR01608")
+					(reference "#PWR01610")
 					(unit 1)
 				)
@@
 		(in_pos_files no)
 		(dnp no)
-		(property "Reference" "#PWR01602"
+		(property "Reference" "#PWR01607"
 			(at 87.63 93.98 0)
 			(hide yes)
@@
 			(project "PingDevKit"
 				(path "/2a5ce3ef-537a-4122-a1be-ef76186bc0d7/a659e729-f286-4529-89a9-b647d33044af"
-					(reference "#PWR01602")
+					(reference "#PWR01607")
 					(unit 1)
 				)
@@
 		(dnp no)
 		(fields_autoplaced yes)
-		(property "Reference" "C1607"
+		(property "Reference" "C1601"
 			(at 63.5 72.3962 0)
 			(show_name no)
@@
 			(project "PingDevKit"
 				(path "/2a5ce3ef-537a-4122-a1be-ef76186bc0d7/a659e729-f286-4529-89a9-b647d33044af"
-					(reference "C1607")
+					(reference "C1601")
 					(unit 1)
 				)
@@
 		(dnp no)
 		(fields_autoplaced yes)
-		(property "Reference" "C1605"
+		(property "Reference" "C1606"
 			(at 125.73 80.0162 0)
 			(show_name no)
@@
 			(project "PingDevKit"
 				(path "/2a5ce3ef-537a-4122-a1be-ef76186bc0d7/a659e729-f286-4529-89a9-b647d33044af"
-					(reference "C1605")
+					(reference "C1606")
 					(unit 1)
 				)
@@
 		(in_pos_files yes)
 		(dnp no)
-		(property "Reference" "#PWR01614"
+		(property "Reference" "#PWR01615"
 			(at 179.07 67.31 0)
 			(hide yes)
@@
 			(project "PingDevKit"
 				(path "/2a5ce3ef-537a-4122-a1be-ef76186bc0d7/a659e729-f286-4529-89a9-b647d33044af"
-					(reference "#PWR01614")
+					(reference "#PWR01615")
 					(unit 1)
 				)
@@
 		(in_pos_files yes)
 		(dnp no)
-		(property "Reference" "#PWR01611"
+		(property "Reference" "#PWR01602"
 			(at 44.45 49.53 0)
 			(hide yes)
@@
 			(project "PingDevKit"
 				(path "/2a5ce3ef-537a-4122-a1be-ef76186bc0d7/a659e729-f286-4529-89a9-b647d33044af"
-					(reference "#PWR01611")
+					(reference "#PWR01602")
 					(unit 1)
 				)
@@
 		(in_pos_files yes)
 		(dnp no)
-		(property "Reference" "#PWR01612"
+		(property "Reference" "#PWR01603"
 			(at 44.45 66.04 0)
 			(hide yes)
@@
 			(project "PingDevKit"
 				(path "/2a5ce3ef-537a-4122-a1be-ef76186bc0d7/a659e729-f286-4529-89a9-b647d33044af"
-					(reference "#PWR01612")
+					(reference "#PWR01603")
 					(unit 1)
 				)
@@
 		(in_pos_files no)
 		(dnp no)
-		(property "Reference" "#PWR01616"
+		(property "Reference" "#PWR01617"
 			(at 181.61 153.67 0)
 			(hide yes)
@@
 			(project "PingDevKit"
 				(path "/2a5ce3ef-537a-4122-a1be-ef76186bc0d7/a659e729-f286-4529-89a9-b647d33044af"
-					(reference "#PWR01616")
+					(reference "#PWR01617")
 					(unit 1)
 				)
@@
 		(in_pos_files yes)
 		(dnp no)
-		(property "Reference" "#PWR01613"
+		(property "Reference" "#PWR01609"
 			(at 102.87 88.9 0)
 			(hide yes)
@@
 			(project "PingDevKit"
 				(path "/2a5ce3ef-537a-4122-a1be-ef76186bc0d7/a659e729-f286-4529-89a9-b647d33044af"
-					(reference "#PWR01613")
+					(reference "#PWR01609")
 					(unit 1)
 				)
@@
 		(in_pos_files no)
 		(dnp no)
-		(property "Reference" "#PWR01605"
+		(property "Reference" "#PWR01611"
 			(at 130.81 137.16 0)
 			(hide yes)
@@
 			(project "PingDevKit"
 				(path "/2a5ce3ef-537a-4122-a1be-ef76186bc0d7/a659e729-f286-4529-89a9-b647d33044af"
-					(reference "#PWR01605")
+					(reference "#PWR01611")
 					(unit 1)
 				)
@@
 		(dnp no)
 		(fields_autoplaced yes)
-		(property "Reference" "C1603"
+		(property "Reference" "C1604"
 			(at 109.22 72.3962 0)
 			(show_name no)
@@
 			(project "PingDevKit"
 				(path "/2a5ce3ef-537a-4122-a1be-ef76186bc0d7/a659e729-f286-4529-89a9-b647d33044af"
-					(reference "C1603")
+					(reference "C1604")
 					(unit 1)
 				)
@@
 		(in_pos_files yes)
 		(dnp no)
-		(property "Reference" "#PWR01615"
+		(property "Reference" "#PWR01604"
 			(at 60.96 73.66 0)
 			(hide yes)
@@
 			(project "PingDevKit"
 				(path "/2a5ce3ef-537a-4122-a1be-ef76186bc0d7/a659e729-f286-4529-89a9-b647d33044af"
-					(reference "#PWR01615")
+					(reference "#PWR01604")
 					(unit 1)
 				)
@@
 		(dnp no)
 		(fields_autoplaced yes)
-		(property "Reference" "C1606"
+		(property "Reference" "C1607"
 			(at 182.88 115.5762 0)
 			(show_name no)
@@
 			(project "PingDevKit"
 				(path "/2a5ce3ef-537a-4122-a1be-ef76186bc0d7/a659e729-f286-4529-89a9-b647d33044af"
-					(reference "C1606")
+					(reference "C1607")
 					(unit 1)
 				)
@@
 		(in_pos_files no)
 		(dnp no)
-		(property "Reference" "#PWR01607"
+		(property "Reference" "#PWR01616"
 			(at 180.34 128.27 0)
 			(hide yes)
@@
 			(project "PingDevKit"
 				(path "/2a5ce3ef-537a-4122-a1be-ef76186bc0d7/a659e729-f286-4529-89a9-b647d33044af"
-					(reference "#PWR01607")
+					(reference "#PWR01616")
 					(unit 1)
 				)
@@
 		(in_pos_files no)
 		(dnp no)
-		(property "Reference" "#PWR01618"
+		(property "Reference" "#PWR01612"
 			(at 154.94 138.43 0)
 			(hide yes)
@@
 			(project "PingDevKit"
 				(path "/2a5ce3ef-537a-4122-a1be-ef76186bc0d7/a659e729-f286-4529-89a9-b647d33044af"
-					(reference "#PWR01618")
+					(reference "#PWR01612")
 					(unit 1)
 				)
@@
 		(dnp no)
 		(fields_autoplaced yes)
-		(property "Reference" "C1602"
+		(property "Reference" "C1603"
 			(at 93.98 72.3962 0)
 			(show_name no)
@@
 			(project "PingDevKit"
 				(path "/2a5ce3ef-537a-4122-a1be-ef76186bc0d7/a659e729-f286-4529-89a9-b647d33044af"
-					(reference "C1602")
+					(reference "C1603")
 					(unit 1)
 				)
@@
 		(in_pos_files no)
 		(dnp no)
-		(property "Reference" "#PWR01606"
+		(property "Reference" "#PWR01613"
 			(at 160.02 138.43 0)
 			(hide yes)
@@
 			(project "PingDevKit"
 				(path "/2a5ce3ef-537a-4122-a1be-ef76186bc0d7/a659e729-f286-4529-89a9-b647d33044af"
-					(reference "#PWR01606")
+					(reference "#PWR01613")
 					(unit 1)
 				)
@@
 		(in_pos_files no)
 		(dnp no)
-		(property "Reference" "#PWR01603"
+		(property "Reference" "#PWR01606"
 			(at 76.2 85.09 0)
 			(hide yes)
@@
 			(project "PingDevKit"
 				(path "/2a5ce3ef-537a-4122-a1be-ef76186bc0d7/a659e729-f286-4529-89a9-b647d33044af"
-					(reference "#PWR01603")
+					(reference "#PWR01606")
 					(unit 1)
 				)
@@
 		(dnp no)
 		(fields_autoplaced yes)
-		(property "Reference" "C1604"
+		(property "Reference" "C1605"
 			(at 125.73 72.3962 0)
 			(show_name no)
@@
 			(project "PingDevKit"
 				(path "/2a5ce3ef-537a-4122-a1be-ef76186bc0d7/a659e729-f286-4529-89a9-b647d33044af"
-					(reference "C1604")
+					(reference "C1605")
 					(unit 1)
 				)
@@
 		(in_pos_files no)
 		(dnp no)
-		(property "Reference" "#PWR01610"
+		(property "Reference" "#PWR01601"
 			(at 44.45 35.56 0)
 			(hide yes)
@@
 			(project "PingDevKit"
 				(path "/2a5ce3ef-537a-4122-a1be-ef76186bc0d7/a659e729-f286-4529-89a9-b647d33044af"
-					(reference "#PWR01610")
+					(reference "#PWR01601")
 					(unit 1)
 				)
@@
 		(in_pos_files no)
 		(dnp no)
-		(property "Reference" "#PWR01617"
+		(property "Reference" "#PWR01618"
 			(at 198.12 153.67 0)
 			(hide yes)
@@
 			(project "PingDevKit"
 				(path "/2a5ce3ef-537a-4122-a1be-ef76186bc0d7/a659e729-f286-4529-89a9-b647d33044af"
-					(reference "#PWR01617")
+					(reference "#PWR01618")
 					(unit 1)
 				)
@@
 		(dnp no)
 		(fields_autoplaced yes)
-		(property "Reference" "C1601"
+		(property "Reference" "C1602"
 			(at 78.74 72.3962 0)
 			(show_name no)
@@
 			(project "PingDevKit"
 				(path "/2a5ce3ef-537a-4122-a1be-ef76186bc0d7/a659e729-f286-4529-89a9-b647d33044af"
-					(reference "C1601")
+					(reference "C1602")
 					(unit 1)
 				)
@@
 		(in_pos_files no)
 		(dnp no)
-		(property "Reference" "#PWR01609"
+		(property "Reference" "#PWR01614"
 			(at 163.83 138.43 0)
 			(hide yes)
@@
 			(project "PingDevKit"
 				(path "/2a5ce3ef-537a-4122-a1be-ef76186bc0d7/a659e729-f286-4529-89a9-b647d33044af"
-					(reference "#PWR01609")
+					(reference "#PWR01614")
 					(unit 1)
 				)
@@
 		(in_pos_files no)
 		(dnp no)
-		(property "Reference" "#PWR01601"
+		(property "Reference" "#PWR01605"
 			(at 60.96 85.09 0)
 			(hide yes)
@@
 			(project "PingDevKit"
 				(path "/2a5ce3ef-537a-4122-a1be-ef76186bc0d7/a659e729-f286-4529-89a9-b647d33044af"
-					(reference "#PWR01601")
+					(reference "#PWR01605")
 					(unit 1)
 				)
@@
 		(in_pos_files no)
 		(dnp no)
-		(property "Reference" "#PWR01604"
+		(property "Reference" "#PWR01608"
 			(at 91.44 85.09 0)
 			(hide yes)
@@
 			(project "PingDevKit"
 				(path "/2a5ce3ef-537a-4122-a1be-ef76186bc0d7/a659e729-f286-4529-89a9-b647d33044af"
-					(reference "#PWR01604")
+					(reference "#PWR01608")
 					(unit 1)
 				)

Commit message: fixing some errors
Parts:
- R1604: footprint BR_Passives:C_0402_1005Metric-minimized -> BR_Passives:R_0402_1005Metric-minimized
Changed lines of the file:
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@@
 			)
 		)
-		(property "Footprint" "BR_Passives:C_0402_1005Metric-minimized"
+		(property "Footprint" "BR_Passives:R_0402_1005Metric-minimized"
 			(at 179.07 -6.35 0)
 			(hide yes)

Commit message: getting really close to final
Parts:
- R1603: footprint BR_Passives:C_0402_1005Metric-minimized -> BR_Passives:R_0402_1005Metric-minimized
Changed lines of the file:
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@@
 			)
 		)
-		(property "Footprint" "BR_Passives:C_0402_1005Metric-minimized"
+		(property "Footprint" "BR_Passives:R_0402_1005Metric-minimized"
 			(at 130.81 48.26 0)
 			(hide yes)
