File: 5v_ldo.kicad_sch (KiCad schematic)
At the start: 5 parts, among them U1401 MG78L05T3

Commit message: more work
Parts:
- C1402: symbol BR_Capacitors_0201:C_0201_100nF_25V_X7R_10% -> BR_Capacitors_0201:C_0201_100nF_25V_X5R_10%
- TP1401: value 5V_RX -> TP_RING_TH
- TP1402: value GND -> TP_RING_TH
Connections:
- net VOUT renamed 5V
Other:
- note added: "7V Input"
- moved on the sheet: TP1401, TP1402

Commit message: more work
Parts:
- removed C1401: 330nF 16V, BR_Passives:C_0402_1005Metric-minimized, symbol BR_Capacitors_0402:C_0402_330nF_16V_X7R_10%
- removed C1402: 100nF 25V, BR_Passives:C_0201_0603Metric-minimized, symbol BR_Capacitors_0201:C_0201_100nF_25V_X5R_10%
- removed TP1401, TP1402: TP_RING_TH, BR_Connectors:TEST-TH_BD2.54-P1.4_RED, symbol BR_Connectors:TP_Ring_PTH
- removed U1401: MG78L05T3, BR_SOT:SOT-23, symbol BR_IC_Regulators:MG78L05T3
