File: 7v_boost.kicad_sch (KiCad schematic)
At the start: 11 parts, among them U1301 LM27313XMFX/NOPB

Commit message: more work
Parts:
- added NT1301: Net_Tie_0201, BR_Virtual_Parts:Net_Tie_0201_1608Metric, symbol BR_Virtual_Parts:Net_Tie_0201
- L1301: value 4u7 1.6A -> L_AWP_252012FW-4R7M
- TP1301: value 7V -> TP_RING_TH
- TP1302: value GND -> TP_RING_TH
Connections:
- net GND: now also NT1301.2; no longer C1301.2, C1303.2, R1302.2, U1301.2 (GND)
- net VOUT renamed 7V
- new net PGND: C1301.2, C1303.2, NT1301.1, R1302.2, U1301.2 (GND)
Other:
- note added: "5V Input"
- moved on the sheet: C1303, TP1301, TP1302

Commit message: more work
Parts:
- R1303: value 62k -> 105k; symbol BR_Resistors_0402:R_0402_62k -> BR_Resistors_0402:R_0402_105k; BRE Number BRE-000361 -> BRE-001545; JLCPCB Part Num C137950 -> C2933067; Manufacturer YAGEO -> FOJAN; Manufacturer Part Num RC0402FR-0762KL -> FRC0402F1053TS; Supplier 1 DigiKey -> (none); Supplier 2 DigiKey -> (none); Supplier 3 JLCPCB -> (none); Supplier Part Num 1 311-62.0KLRCT-ND -> (none); Supplier Part Num 2 311-62.0KLRTR-ND -> (none); Supplier Part Num 3 C137950 -> (none)
Connections:
- net 7V renamed 11V
Other:
- note added: "* Vref = 1.23V * FB resistor to GND recommended as 13k3 * 11V means FB resistor to output should be 105k6 * 105k and 13k3 yields 10.9V"
- note removed: "R1401 recommended to be 13.3k R1402 = R1401 * (Vout/1.23 - 1) = 62.3k"
Changed lines of the file:
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@@
 		)
 	)
-	(text "R1401 recommended to be 13.3k\nR1402 = R1401 * (Vout/1.23 - 1)\n= 62.3k"
+	(text "* Vref = 1.23V\n* FB resistor to GND recommended as 13k3\n* 11V means FB resistor to output should be 105k6\n* 105k and 13k3 yields 10.9V\n"
 		(exclude_from_sim no)
-		(at 134.62 61.722 0)
+		(at 149.606 68.072 0)
 		(effects
 			(font
@@
 		)
 	)
-	(hierarchical_label "7V"
+	(hierarchical_label "11V"
 		(shape output)
 		(at 25.4 60.96 180)
@@
 			)
 		)
-		(property "Value" "7V"
+		(property "Value" "11V"
 			(at 38.1 57.404 0)
 			(show_name no)
@@
 	)
 	(symbol
-		(lib_id "BR_Resistors_0402:R_0402_62k")
+		(lib_id "BR_Resistors_0402:R_0402_105k")
 		(at 116.84 69.85 90)
 		(unit 1)
@@
 			)
 		)
-		(property "Value" "62k"
-			(at 116.84 67.056 90)
-			(show_name no)
-			(do_not_autoplace no)
-			(effects
-				(font
-					(size 1.27 1.27)
-				)
+		(property "Value" "105k"
+			(at 118.364 67.056 90)
+			(show_name no)
+			(do_not_autoplace no)
+			(effects
+				(font
+					(size 1.27 1.27)
+				)
+				(justify left)
 			)
 		)
@@
 			)
 		)
-		(property "Datasheet" "https://www.yageo.com/upload/media/product/productsearch/datasheet/rchip/PYu-RC_Group_51_RoHS_L_12.pdf"
+		(property "Datasheet" "https://wmsc.lcsc.com/wmsc/upload/file/pdf/v2/lcsc/2308241947_FOJAN-FRC0402F1053TS_C2933067.pdf"
 			(at 43.18 69.85 0)
 			(hide yes)
@@
 			)
 		)
-		(property "Description" "62k 1% 100ppm 62.5mW Thick Film Resistor 0402"
+		(property "Description" "105k 1% 100ppm 62.5mW Thick Film Resistor 0402"
+			(at 53.34 69.85 0)
+			(hide yes)
+			(show_name no)
+			(do_not_autoplace no)
+			(effects
+				(font
+					(size 1.27 1.27)
+				)
+				(justify left)
+			)
+		)
+		(property "Manufacturer" "FOJAN"
 			(at 45.72 69.85 0)
 			(hide yes)
@@
 			)
 		)
-		(property "Manufacturer" "YAGEO"
+		(property "Manufacturer Part Num" "FRC0402F1053TS"
 			(at 48.26 69.85 0)
 			(hide yes)
@@
 			)
 		)
-		(property "Manufacturer Part Num" "RC0402FR-0762KL"
+		(property "BRE Number" "BRE-001545"
 			(at 50.8 69.85 0)
 			(hide yes)
@@
 			)
 		)
-		(property "BRE Number" "BRE-000361"
-			(at 53.34 69.85 0)
-			(hide yes)
-			(show_name no)
-			(do_not_autoplace no)
-			(effects
-				(font
-					(size 1.27 1.27)
-				)
-				(justify left)
-			)
-		)
-		(property "Supplier 1" "DigiKey"
+		(property "JLCPCB Part Num" "C2933067"
 			(at 55.88 69.85 0)
-			(hide yes)
-			(show_name no)
-			(do_not_autoplace no)
-			(effects
-				(font
-					(size 1.27 1.27)
-				)
-				(justify left)
-			)
-		)
-		(property "Supplier Part Num 1" "311-62.0KLRCT-ND"
-			(at 58.42 69.85 0)
-			(hide yes)
-			(show_name no)
-			(do_not_autoplace no)
-			(effects
-				(font
-					(size 1.27 1.27)
-				)
-				(justify left)
-			)
-		)
-		(property "Supplier 2" "DigiKey"
-			(at 60.96 69.85 0)
-			(hide yes)
-			(show_name no)
-			(do_not_autoplace no)
-			(effects
-				(font
-					(size 1.27 1.27)
-				)
-				(justify left)
-			)
-		)
-		(property "Supplier Part Num 2" "311-62.0KLRTR-ND"
-			(at 63.5 69.85 0)
-			(hide yes)
-			(show_name no)
-			(do_not_autoplace no)
-			(effects
-				(font
-					(size 1.27 1.27)
-				)
-				(justify left)
-			)
-		)
-		(property "Supplier 3" "JLCPCB"
-			(at 66.04 69.85 0)
-			(hide yes)
-			(show_name no)
-			(do_not_autoplace no)
-			(effects
-				(font
-					(size 1.27 1.27)
-				)
-				(justify left)
-			)
-		)
-		(property "Supplier Part Num 3" "C137950"
-			(at 68.58 69.85 0)
-			(hide yes)
-			(show_name no)
-			(do_not_autoplace no)
-			(effects
-				(font
-					(size 1.27 1.27)
-				)
-				(justify left)
-			)
-		)
-		(property "JLCPCB Part Num" "C137950"
-			(at 71.12 69.85 0)
 			(hide yes)
 			(show_name no)
@@
 			)
 		)
-		(property "Value" "7V"
+		(property "Value" "11V"
 			(at 140.97 45.974 0)
 			(show_name no)

Commit message: more work
Parts:
- C1302: value 330pF 50V -> 200pF 50V; symbol BR_Capacitors_0402:C_0402_330pF_50V_C0G_5% -> BR_Capacitors_0402:C_0402_200pF_50V_C0G_5%; BRE Number BRE-001236 -> BRE-001222; JLCPCB Part Num C107006 -> C325462; Manufacturer Part Num CC0402JRNPO9BN331 -> CC0402JRNPO9BN201
Other:
- note added: "* Vref = 1.23V * FB resistor to GND recommended as 13k3 * 11V means FB resistor to output should be 105k6 * 105k and 13k3 yields 10.9V * F3db of C1302 and R1303 should be ~ 8 kHz"
- note removed: "* Vref = 1.23V * FB resistor to GND recommended as 13k3 * 11V means FB resistor to output should be 105k6 * 105k and 13k3 yields 10.9V"
Changed lines of the file:
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@@
 		)
 	)
-	(text "* Vref = 1.23V\n* FB resistor to GND recommended as 13k3\n* 11V means FB resistor to output should be 105k6\n* 105k and 13k3 yields 10.9V\n"
+	(text "* Vref = 1.23V\n* FB resistor to GND recommended as 13k3\n* 11V means FB resistor to output should be 105k6\n* 105k and 13k3 yields 10.9V\n* F3db of C1302 and R1303 should be ~ 8 kHz\n"
 		(exclude_from_sim no)
 		(at 149.606 68.072 0)
@@
 	)
 	(symbol
-		(lib_id "BR_Capacitors_0402:C_0402_330pF_50V_C0G_5%")
+		(lib_id "BR_Capacitors_0402:C_0402_200pF_50V_C0G_5%")
 		(at 116.84 78.74 90)
 		(unit 1)
@@
 			)
 		)
-		(property "Value" "330pF 50V"
-			(at 116.84 75.946 90)
-			(show_name no)
-			(do_not_autoplace no)
-			(effects
-				(font
-					(size 1.27 1.27)
-				)
+		(property "Value" "200pF 50V"
+			(at 124.46 76.2 90)
+			(show_name no)
+			(do_not_autoplace no)
+			(effects
+				(font
+					(size 1.27 1.27)
+				)
+				(justify left)
 			)
 		)
@@
 			)
 		)
-		(property "Datasheet" "https://lcsc.com/datasheet/lcsc_datasheet_2506131730_YAGEO-CC0402JRNPO9BN331_C107006.pdf"
+		(property "Datasheet" "https://jlcpcb.com/api/file/downloadByFileSystemAccessId/8588946632188022784"
 			(at 43.18 78.74 0)
 			(hide yes)
@@
 			)
 		)
-		(property "Description" "330pF 50V C0G 5% Ceramic Capacitor 0402"
+		(property "Description" "200pF 50V C0G 5% Ceramic Capacitor 0402"
 			(at 45.72 78.74 0)
 			(hide yes)
@@
 			)
 		)
-		(property "Manufacturer Part Num" "CC0402JRNPO9BN331"
+		(property "Manufacturer Part Num" "CC0402JRNPO9BN201"
 			(at 50.8 78.74 0)
 			(hide yes)
@@
 			)
 		)
-		(property "BRE Number" "BRE-001236"
+		(property "BRE Number" "BRE-001222"
 			(at 53.34 78.74 0)
 			(hide yes)
@@
 			)
 		)
-		(property "JLCPCB Part Num" "C107006"
+		(property "JLCPCB Part Num" "C325462"
 			(at 55.88 78.74 0)
 			(hide yes)
@@
 		(in_pos_files yes)
 		(dnp no)
-		(fields_autoplaced yes)
 		(property "Reference" "NT1301"
-			(at 97.79 96.52 90)
-			(hide yes)
+			(at 99.06 99.06 90)
 			(show_name no)
 			(do_not_autoplace no)
@@
 		)
 		(property "Value" "Net_Tie_0201"
-			(at 97.79 99.06 90)
-			(show_name no)
-			(do_not_autoplace no)
+			(at 101.6 99.06 90)
+			(hide yes)
+			(show_name no)
+			(do_not_autoplace no)
