File: PSRAM.kicad_sch (KiCad schematic)
At the start: 6 parts, among them J901 FPGA, U901 S27KL0642DPBHB023

Commit message: starting to incorporate todos
Parts:
- removed J901: FPGA, BR_Connectors:HDR-SMD_20P-P2.54-V-M-R2-C10-S7.5, symbol BR_Connectors_Header:Header_Pin_02x10_2.54mm_Vert_PTH
Connections:
- no-connect marks 5 -> 0

Commit message: more work
Parts:
- C901: JLCPCB Part Num C23692972 -> C528974
Changed lines of the file:
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@@
 	)
 	(label "OCTOSPI1.RST"
-		(at 78.74 58.42 0)
+		(at 92.71 58.42 180)
 		(effects
 			(font
 				(size 1.27 1.27)
 			)
-			(justify left bottom)
+			(justify right bottom)
 		)
 	)
@@
 			)
 		)
-		(property "JLCPCB Part Num" "C23692972"
+		(property "JLCPCB Part Num" "C528974"
 			(at 135.89 7.62 0)
 			(hide yes)
