File: PingDevKit.kicad_sch (KiCad schematic)
At the start: 46 parts, among them J102 PGM, J103 ETH, J104 RX, J105 ETH, J106 SYNC, J107 TX-, J108 RX+, J109 TX+, J110 RX-, J111 XDCR, J112 LABEL, J113 XDCR, J22 PWR IN, J401 RX, J501 TX, Q101 DMP6023LSS-13, T101 B65655B0010X000, U101 LIS2DH12TR

Commit message: more work
Connections:
- net TX/DAMP: now reaches J501.16 (Pin_16)
- net DTX_SD renamed TX_DSD
- net MCU/GPIO_D4 renamed TX_DAMP
- no-connect marks 15 -> 14
Other:
- sheet TX ports: added DAMP; removed none
Changed lines of the file:
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@@
 	)
 	(no_connect
-		(at 379.73 170.18)
-	)
-	(no_connect
 		(at 473.71 167.64)
 	)
@@
 	(wire
 		(pts
+			(xy 379.73 170.18) (xy 392.43 170.18)
+		)
+		(stroke
+			(width 0)
+			(type default)
+		)
+	)
+	(wire
+		(pts
 			(xy 68.58 87.63) (xy 68.58 90.17)
 		)
@@
 		)
 	)
+	(label "TX_DAMP"
+		(at 344.17 170.18 0)
+		(effects
+			(font
+				(size 1.27 1.27)
+			)
+			(justify left bottom)
+		)
+	)
 	(label "SONAR+"
 		(at 496.57 133.35 180)
@@
 		)
 	)
-	(label "DTX_SD"
+	(label "TX_DSD"
 		(at 344.17 152.4 0)
 		(effects
@@
 	)
 	(label "TX_EN"
-		(at 345.44 167.64 0)
+		(at 344.17 167.64 0)
 		(effects
 			(font
@@
 			(effects
 				(font
+					(size 1.27 1.27)
+				)
+				(justify left)
+			)
+		)
+		(pin "DAMP" input
+			(at 392.43 170.18 180)
+			(effects
+				(font

Commit message: more work
Parts:
- added D301: DEBUG, BR_Optoelectronics:LED_0603_1608Metric, symbol BR_Optoelectronic:ORH-G36G
- added R303: 3k, BR_Passives:R_0201_0603Metric-minimized, symbol BR_Resistors_0201:R_0201_3k
Connections:
- net GND: now also D301.1
- new net: D301.2, R303.2
- new net DEBUG_LED: R303.1
- no-connect marks 14 -> 15
Other:
- sheet MCU ports: added ADC12_INP3, GPIO_F7; removed none
- sheet PSRAM ports: added GND; removed none
- sheet Power ports: added RX_10V; removed none
- sheet RX ports: added 10V; removed none
- moved on the sheet: C104, J103, J105, J106, J107, J108, J109, J110, J111, J112, J113, J401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

Commit message: more work
Other:
- sheet Ethernet ports: added none; removed PHY_REF_CLK
- sheet MCU ports: added GPIO_H3, GPIO_H4, GPIO_H9; removed PHY_REF_CLK, PHY_nRST, VTX_EN, VTX_MODE
- sheet Power ports: added none; removed VTX_MODE

Commit message: more work
Parts:
- removed TP103, TP104: TP_RING_TH, BR_Connectors:TEST-TH_BD2.54-P1.4_RED, symbol BR_Connectors:TP_Ring_PTH
- added TP101, TP103, TP104: value, BR_Virtual_Parts:TP_PROBE_TIP_WITH_GND, symbol BR_Virtual_Parts:TP_Probe_Tip_0.8mm_Hole_with_GND
Connections:
- net GND: now also TP101.2 (GND), TP103.2 (GND), TP104.2 (GND)
- net RX_SIG_AFE: now also TP101.1
- net SONAR+: now also TP103.1
- net SONAR-: now also TP104.1

Commit message: more work
Parts:
- renumbered C105 to C104, C106 to C105, C107 to C106, C108 to C107, C109 to C108, C110 to C109, C113 to C110, C114 to C111, C104 to C112, D301 to D102, J22 to J101, J106 to J103, J501 to J105, J401 to J106, J112 to J107, J105 to J108, J107 to J110, J108 to J111, J110 to J112, J103 to J113, J113 to J114, J111 to J115, R103 to R101, R303 to R102, R104 to R103, R114 to R104, R101 to R105, R102 to R106, TP102 to TP101, TP101 to TP102

Commit message: more work
Connections:
- net TX/PWM_B: no longer R104.1
Changed lines of the file:
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@@
-	)
-	(junction
-		(at 384.81 184.15)
-		(diameter 0)
-		(color 0 0 0 0)
 	)
 	(junction
@@
 	(wire
 		(pts
-			(xy 384.81 184.15) (xy 391.16 184.15)
+			(xy 379.73 184.15) (xy 391.16 184.15)
 		)
 		(stroke
@@
 	(wire
 		(pts
-			(xy 384.81 175.26) (xy 384.81 184.15)
-		)
-		(stroke
-			(width 0)
-			(type default)
-		)
-	)
-	(wire
-		(pts
 			(xy 228.6 69.85) (xy 290.83 69.85)
 		)
@@
 		)
 		(stroke
-			(width 0)
-			(type default)
-		)
-	)
-	(wire
-		(pts
-			(xy 379.73 184.15) (xy 384.81 184.15)
-		)
-		(stroke

Commit message: more work
Parts:
- removed R104: 10k, BR_Passives:C_0402_1005Metric-minimized, symbol BR_Resistors_0402:R_0402_10k
Connections:
- net MCU/GPIO_H4: now also J104.6 (Pin_6)
- no-connect marks 15 -> 13
Other:
- sheet MCU ports: added none; removed ADC12_INP12

Commit message: work
Parts:
- removed TP101: TP_RING_TH, BR_Connectors:TEST-TH_BD2.54-P1.4_RED, symbol BR_Connectors:TP_Ring_PTH
- added TP101: VTX, BR_Virtual_Parts:TP_SQUARE_TH_1mm, symbol BR_Virtual_Parts:TP_SQUARE_TH_1mm
- added TP105: TX_SIG, BR_Virtual_Parts:TP_PROBE_TIP_WITH_GND, symbol BR_Virtual_Parts:TP_Probe_Tip_0.8mm_Hole_with_GND
- added TP106: TX_EN, BR_Virtual_Parts:TP_PROBE_TIP_WITH_GND, symbol BR_Virtual_Parts:TP_Probe_Tip_0.8mm_Hole_with_GND
- added TP107, TP108: GND, BR_Connectors:TEST-TH_BD2.54-P1.4_RED, symbol BR_Connectors:TP_Ring_PTH
- added TP109: 5V, BR_Virtual_Parts:TP_SQUARE_TH_1mm, symbol BR_Virtual_Parts:TP_SQUARE_TH_1mm
- added TP110: RX_10V, BR_Virtual_Parts:TP_SQUARE_TH_1mm, symbol BR_Virtual_Parts:TP_SQUARE_TH_1mm
- added TP111: RX_5V, BR_Virtual_Parts:TP_SQUARE_TH_1mm, symbol BR_Virtual_Parts:TP_SQUARE_TH_1mm
- added TP112: 3V3, BR_Virtual_Parts:TP_SQUARE_TH_1mm, symbol BR_Virtual_Parts:TP_SQUARE_TH_1mm
- TP102: value value -> RX_SIG
- TP103: value value -> SONAR+
- TP104: value value -> SONAR-
Connections:
- net 3V3: now also TP112.1
- net 5V: now also TP109.1
- net GND: now also TP105.2 (GND), TP106.2 (GND), TP107.1, TP108.1
- net RX_10V: now also TP110.1
- net RX_5V: now also TP111.1
- net RX_SIG: now also TP102.1
- net RX_SIG_AFE: no longer TP102.1
- net TX_EN: now also TP106.1
- net TX_SIG: now also TP105.1
- net VTX: now also TP101.1
Other:
- moved on the sheet: TP102
