File: digital_drive.kicad_sch (KiCad schematic)
At the start: 19 parts, among them U1501 EPC23104ENGRT, U1502 EPC23104ENGRT

Commit message: more work
Connections:
- net SD1 is gone; now on net SD0: U1502.3 (SD)
Other:
- moved on the sheet: C1501, C1502, C1503, C1504, C1505, C1506, C1507, C1508, C1509, C1510, R1502, R1503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

Commit message: more work
Parts:
- C1501, C1506: JLCPCB Part Num C23692972 -> C528974
- NT1501: value NetTie-2_0.18mm -> Net Tie
- TP1501: value PWM_A -> TP_RING_TH
- TP1502: value PWM_B -> TP_RING_TH
Connections:
- net SD0 renamed SD
Other:
- moved on the sheet: C1509, C1510

Commit message: refactoring interconnects to simplify busses
Parts:
- added R1501: 1k, BR_Passives:C_0402_1005Metric-minimized, symbol BR_Resistors_0402:R_0402_1k
Connections:
- net SD: now also R1501.1
- new net 3V3: R1501.2

Commit message: more work
Parts:
- renumbered C1506 to C1502, C1502 to C1503, C1505 to C1504, C1503 to C1505, C1504 to C1506, C1510 to C1508, C1508 to C1509, C1509 to C1510, R1502 to R1501, R1503 to R1502, R1504 to R1503, R1505 to R1504, R1501 to R1505

Commit message: more work
Parts:
- removed TP1501, TP1502: TP_RING_TH, BR_Connectors:TEST-TH_BD2.54-P1.4_RED, symbol BR_Connectors:TP_Ring_PTH
- R1505: symbol BR_Resistors_0402:R_0402_1k -> BR_Resistors_0402:R_0402_10k; BRE Number BRE-000311 -> BRE-000292; JLCPCB Part Num C106235 -> C144807; Manufacturer Part Num RC0402FR-071KL -> AC0402FR-0710KL; Supplier Part Num 1 311-1.00KLRCT-ND -> YAG3436CT-ND; Supplier Part Num 2 311-1.00KLRTR-ND -> YAG3436TR-ND; Supplier Part Num 3 C106235 -> C144807
Connections:
- net 3V3: no longer R1505.2
- net 5V: now also R1505.2

Commit message: more work
Connections:
- net VTX renamed VRAIL
Changed lines of the file:
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@@
 		)
 	)
-	(hierarchical_label "VTX"
+	(hierarchical_label "VRAIL"
 		(shape input)
 		(at 77.47 25.4 180)
@@
 			)
 		)
-		(property "Value" "VTX"
+		(property "Value" "VRAIL"
 			(at 95.25 21.844 0)
 			(show_name no)
@@
 			)
 		)
-		(property "Value" "VTX"
+		(property "Value" "VRAIL"
 			(at 130.81 132.334 0)
 			(show_name no)
@@
 			)
 		)
-		(property "Value" "VTX"
+		(property "Value" "VRAIL"
 			(at 130.81 76.454 0)
 			(show_name no)

Commit message: fixing some errors
Parts:
- R1505: footprint BR_Passives:C_0402_1005Metric-minimized -> BR_Passives:R_0402_1005Metric-minimized
Changed lines of the file:
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@@
 			)
 		)
-		(property "Footprint" "BR_Passives:C_0402_1005Metric-minimized"
+		(property "Footprint" "BR_Passives:R_0402_1005Metric-minimized"
 			(at 22.86 69.85 0)
 			(hide yes)
