File: ethernet.kicad_sch (KiCad schematic)
At the start: 26 parts, among them T701 TRANSFORMER ARRAY, U701 ETHERNET

Commit message: more work
Parts:
- C703, C709, C710: JLCPCB Part Num C23692972 -> C528974
- C704, C707, C708: symbol BR_Capacitors_0201:C_0201_100nF_25V_X7R_10% -> BR_Capacitors_0201:C_0201_100nF_25V_X5R_10%
- T701: value TRANSFORMER ARRAY -> HR641680E
- U701: value ETHERNET -> DP83825IRMQR
Other:
- moved on the sheet: C701, C702, C703, C704, C705, C706, C707, C708, C709, C710, C711, C712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

Commit message: more work
Connections:
- net RD_N renamed MDI.RX-
- net RD_P renamed MDI.RX+
- net TD_N renamed MDI.TX-
- net TD_P renamed MDI.TX+
Other:
- moved on the sheet: C701, C702, C703, C704, C705, C706, C707, C708, C709, C710, C711, C712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

Commit message: more work
Connections:
- net PHY_REF_CLK renamed MAC.REF_CLK
Changed lines of the file:
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@@
+	)
+	(bus_entry
+		(at 227.33 269.24)
+		(size -2.54 2.54)
+		(stroke
+			(width 0)
+			(type default)
+		)
 	)
 	(bus_entry
@@
 	(bus
 		(pts
-			(xy 224.79 238.76) (xy 224.79 241.3)
+			(xy 224.79 238.76) (xy 224.79 271.78)
 		)
 		(stroke
@@
 	(wire
 		(pts
-			(xy 302.26 256.54) (xy 302.26 261.62)
+			(xy 302.26 256.54) (xy 302.26 269.24)
 		)
 		(stroke
@@
 	(wire
 		(pts
+			(xy 227.33 269.24) (xy 302.26 269.24)
+		)
+		(stroke
+			(width 0)
+			(type default)
+		)
+	)
+	(wire
+		(pts
 			(xy 414.02 184.15) (xy 414.02 173.99)
 		)
@@
 	(bus
 		(pts
-			(xy 224.79 241.3) (xy 214.63 241.3)
+			(xy 224.79 271.78) (xy 214.63 271.78)
 		)
 		(stroke
@@
 		)
 	)
+	(label "MAC.REF_CLK"
+		(at 283.21 269.24 0)
+		(effects
+			(font
+				(size 1.27 1.27)
+			)
+			(justify left bottom)
+		)
+	)
 	(label "MDI{100BASE-T}"
 		(at 356.87 196.85 0)
@@
 			)
 			(justify left bottom)
-		)
-	)
-	(hierarchical_label "PHY_REF_CLK"
-		(shape input)
-		(at 302.26 261.62 270)
-		(effects
-			(font
-				(size 1.27 1.27)
-			)
-			(justify right)
 		)
 	)
@@
 	(hierarchical_label "MAC{RMII}"
 		(shape input)
-		(at 214.63 241.3 180)
-		(effects
-			(font
+		(at 214.63 271.78 180)
+		(effects
+			(font

Commit message: more work
Parts:
- renumbered C711 to C701, C710 to C702, C709 to C703, C707 to C704, C706 to C705, C705 to C706, C704 to C707, C703 to C708, C701 to C709, C708 to C710, C712 to C711, C702 to C712, R711 to R701, R710 to R702, R709 to R703, R708 to R704, R706 to R705, R712 to R706, R705 to R707, R702 to R708, R701 to R709, R707 to R710, R703 to R711, R704 to R712

Commit message: fixing some errors
Parts:
- R701, R702, R703, R704, R708, R709: footprint BR_Passives:C_0402_1005Metric-minimized -> BR_Passives:R_0402_1005Metric-minimized
Changed lines of the file:
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@@
 			)
 		)
-		(property "Footprint" "BR_Passives:C_0402_1005Metric-minimized"
+		(property "Footprint" "BR_Passives:R_0402_1005Metric-minimized"
 			(at 236.22 172.72 0)
 			(hide yes)
@@
 			)
 		)
-		(property "Footprint" "BR_Passives:C_0402_1005Metric-minimized"
+		(property "Footprint" "BR_Passives:R_0402_1005Metric-minimized"
 			(at 251.46 121.92 0)
 			(hide yes)
@@
 			)
 		)
-		(property "Footprint" "BR_Passives:C_0402_1005Metric-minimized"
+		(property "Footprint" "BR_Passives:R_0402_1005Metric-minimized"
 			(at 369.57 171.45 0)
 			(hide yes)
@@
 			)
 		)
-		(property "Footprint" "BR_Passives:C_0402_1005Metric-minimized"
+		(property "Footprint" "BR_Passives:R_0402_1005Metric-minimized"
 			(at 246.38 172.72 0)
 			(hide yes)
@@
 			)
 		)
-		(property "Footprint" "BR_Passives:C_0402_1005Metric-minimized"
+		(property "Footprint" "BR_Passives:R_0402_1005Metric-minimized"
 			(at 408.94 168.91 0)
 			(hide yes)
@@
 			)
 		)
-		(property "Footprint" "BR_Passives:C_0402_1005Metric-minimized"
+		(property "Footprint" "BR_Passives:R_0402_1005Metric-minimized"
 			(at 256.54 172.72 0)
 			(hide yes)

Commit message: getting really close to final
Parts:
- R705, R706, R707, R710, R711, R712: footprint BR_Passives:C_0402_1005Metric-minimized -> BR_Passives:R_0402_1005Metric-minimized
Changed lines of the file:
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@@
 			)
 		)
-		(property "Footprint" "BR_Passives:C_0402_1005Metric-minimized"
+		(property "Footprint" "BR_Passives:R_0402_1005Metric-minimized"
 			(at 369.57 210.82 0)
 			(hide yes)
@@
 			)
 		)
-		(property "Footprint" "BR_Passives:C_0402_1005Metric-minimized"
+		(property "Footprint" "BR_Passives:R_0402_1005Metric-minimized"
 			(at 341.63 173.99 0)
 			(hide yes)
@@
 			)
 		)
-		(property "Footprint" "BR_Passives:C_0402_1005Metric-minimized"
+		(property "Footprint" "BR_Passives:R_0402_1005Metric-minimized"
 			(at 345.44 187.96 0)
 			(hide yes)
@@
 			)
 		)
-		(property "Footprint" "BR_Passives:C_0402_1005Metric-minimized"
+		(property "Footprint" "BR_Passives:R_0402_1005Metric-minimized"
 			(at 347.98 184.15 0)
 			(hide yes)
@@
 			)
 		)
-		(property "Footprint" "BR_Passives:C_0402_1005Metric-minimized"
+		(property "Footprint" "BR_Passives:R_0402_1005Metric-minimized"
 			(at 539.75 213.36 0)
 			(hide yes)
@@
 			)
 		)
-		(property "Footprint" "BR_Passives:C_0402_1005Metric-minimized"
+		(property "Footprint" "BR_Passives:R_0402_1005Metric-minimized"
 			(at 539.75 204.47 0)
 			(hide yes)
