File: fdcan.kicad_sch (KiCad schematic)
At the start: 8 parts, among them U1401 SIT1042A

Commit message: fixing some errors
Parts:
- R1401, R1402: footprint BR_Passives:C_0402_1005Metric-minimized -> BR_Passives:R_0402_1005Metric-minimized
Changed lines of the file:
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@@
 			)
 		)
-		(property "Footprint" "BR_Passives:C_0402_1005Metric-minimized"
+		(property "Footprint" "BR_Passives:R_0402_1005Metric-minimized"
 			(at 177.8 182.88 0)
 			(hide yes)
@@
 			)
 		)
+		(property "Sim.Enable" "0"
+			(at 238.76 182.88 0)
+			(hide yes)
+			(show_name no)
+			(do_not_autoplace no)
+			(effects
+				(font
+					(size 1.27 1.27)
+				)
+			)
+		)
 		(pin "1"
 		)
@@
 			)
 		)
-		(property "Footprint" "BR_Passives:C_0402_1005Metric-minimized"
+		(property "Footprint" "BR_Passives:R_0402_1005Metric-minimized"
 			(at 218.44 193.04 0)
 			(hide yes)
@@
 			)
 		)
+		(property "Sim.Enable" "0"
+			(at 238.76 180.34 0)
+			(hide yes)
+			(show_name no)
+			(do_not_autoplace no)
+			(effects
+				(font
+					(size 1.27 1.27)
+				)
+			)
+		)
 		(pin "1"
 		)
@@
 			)
 		)
+		(property "Sim.Enable" "0"
+			(at 238.76 185.42 0)
+			(hide yes)
+			(show_name no)
+			(do_not_autoplace no)
+			(effects
+				(font
+					(size 1.27 1.27)
+				)
+			)
+		)

Commit message: getting really close to final
Parts:
- TP1401, TP1402, TP1403: footprint BR_Virtual_Parts:TP_SQUARE_TH_1mm -> BR_Virtual_Parts:TP_SQUARE_TH_2mm; symbol BR_Virtual_Parts:TP_SQUARE_TH_1mm -> BR_Virtual_Parts:TP_SQUARE_TH_2mm; BRE Number BRE-000074 -> (none); JLCPCB Part Num C5277086 -> (none); Label LABEL -> (none); Manufacturer ronghe -> (none); Manufacturer Part Num RH-5000 -> (none); Supplier 1 DigiKey -> (none); Supplier 2 Mouser -> (none); Supplier 3 JLCPCB -> (none); Supplier Part Num 3 C5277086 -> (none)
- U1401: JLCPCB Part Num (none) -> C5382546
Changed lines of the file:
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@@
+			)
+		)
+		(property "JLCPCB Part Num" "C5382546"
+			(at 274.32 127 0)
+			(hide yes)
+			(show_name no)
+			(do_not_autoplace no)
+			(effects
+				(font
+					(size 1.27 1.27)
+				)
+				(justify left)
 			)
 		)
@@
 	)
 	(symbol
-		(lib_id "BR_Virtual_Parts:TP_SQUARE_TH_1mm")
+		(lib_id "BR_Virtual_Parts:TP_SQUARE_TH_2mm")
 		(at 238.76 182.88 90)
 		(unit 1)
 		(body_style 1)
-		(exclude_from_sim yes)
+		(exclude_from_sim no)
 		(in_bom no)
 		(on_board yes)
@@
 			)
 		)
-		(property "Footprint" "BR_Virtual_Parts:TP_SQUARE_TH_1mm"
+		(property "Footprint" "BR_Virtual_Parts:TP_SQUARE_TH_2mm"
 			(at 231.394 181.61 0)
 			(hide yes)
@@
 			)
 		)
-		(property "Datasheet" "https://wmsc.lcsc.com/wmsc/upload/file/pdf/v2/lcsc/2307040929_ronghe-RH-5000_C5277086.pdf"
+		(property "Datasheet" ""
 			(at 231.267 182.626 0)
 			(hide yes)
@@
 			)
 		)
-		(property "Description" "test pad through hole"
+		(property "Description" "test pad, through hole"
 			(at 238.76 182.88 0)
 			(hide yes)
@@
 			)
 		)
-		(property "Manufacturer" "ronghe"
+		(property "Manufacturer" ""
 			(at 230.759 184.404 0)
 			(hide yes)
@@
 			)
 		)
-		(property "Manufacturer Part Num" "RH-5000"
+		(property "Manufacturer Part Num" ""
 			(at 231.648 183.134 0)
 			(hide yes)
@@
 			)
 		)
-		(property "BRE Number" "BRE-000074"
-			(at 175.26 182.88 0)
-			(hide yes)
-			(show_name no)
-			(do_not_autoplace no)
-			(effects
-				(font
-					(size 1.27 1.27)
-				)
-				(justify left)
-			)
-		)
-		(property "Supplier 1" "DigiKey"
+		(property "Supplier 1" ""
 			(at 231.14 184.785 0)
 			(hide yes)
@@
 			)
 		)
-		(property "Supplier 2" "Mouser"
+		(property "Supplier 2" ""
 			(at 231.648 184.15 0)
 			(hide yes)
@@
 					(size 1.27 1.27)
 				)
-			)
-		)
-		(property "Supplier 3" "JLCPCB"
-			(at 187.96 182.88 0)
-			(hide yes)
-			(show_name no)
-			(do_not_autoplace no)
-			(effects
-				(font
-					(size 1.27 1.27)
-				)
-				(justify left)
-			)
-		)
-		(property "Supplier Part Num 3" "C5277086"
-			(at 190.5 182.88 0)
-			(hide yes)
-			(show_name no)
-			(do_not_autoplace no)
-			(effects
-				(font
-					(size 1.27 1.27)
-				)
-				(justify left)
-			)
-		)
-		(property "Label" "LABEL"
-			(at 193.04 182.88 0)
-			(hide yes)
-			(show_name no)
-			(do_not_autoplace no)
-			(effects
-				(font
-					(size 1.27 1.27)
-				)
-				(justify left)
-			)
-		)
-		(property "JLCPCB Part Num" "C5277086"
-			(at 195.58 182.88 0)
-			(hide yes)
-			(show_name no)
-			(do_not_autoplace no)
-			(effects
-				(font
-					(size 1.27 1.27)
-				)
-				(justify left)
 			)
 		)
@@
 	)
 	(symbol
-		(lib_id "BR_Virtual_Parts:TP_SQUARE_TH_1mm")
+		(lib_id "BR_Virtual_Parts:TP_SQUARE_TH_2mm")
 		(at 238.76 180.34 90)
 		(unit 1)
 		(body_style 1)
-		(exclude_from_sim yes)
+		(exclude_from_sim no)
 		(in_bom no)
 		(on_board yes)
@@
 			)
 		)
-		(property "Footprint" "BR_Virtual_Parts:TP_SQUARE_TH_1mm"
+		(property "Footprint" "BR_Virtual_Parts:TP_SQUARE_TH_2mm"
 			(at 231.394 179.07 0)
 			(hide yes)
@@
 			)
 		)
-		(property "Datasheet" "https://wmsc.lcsc.com/wmsc/upload/file/pdf/v2/lcsc/2307040929_ronghe-RH-5000_C5277086.pdf"
+		(property "Datasheet" ""
 			(at 231.267 180.086 0)
 			(hide yes)
@@
 			)
 		)
-		(property "Description" "test pad through hole"
+		(property "Description" "test pad, through hole"
 			(at 238.76 180.34 0)
 			(hide yes)
@@
 			)
 		)
-		(property "Manufacturer" "ronghe"
+		(property "Manufacturer" ""
 			(at 230.759 181.864 0)
 			(hide yes)
@@
 			)
 		)
-		(property "Manufacturer Part Num" "RH-5000"
+		(property "Manufacturer Part Num" ""
 			(at 231.648 180.594 0)
 			(hide yes)
@@
 			)
 		)
-		(property "BRE Number" "BRE-000074"
-			(at 175.26 180.34 0)
-			(hide yes)
-			(show_name no)
-			(do_not_autoplace no)
-			(effects
-				(font
-					(size 1.27 1.27)
-				)
-				(justify left)
-			)
-		)
-		(property "Supplier 1" "DigiKey"
+		(property "Supplier 1" ""
 			(at 231.14 182.245 0)
 			(hide yes)
@@
 			)
 		)
-		(property "Supplier 2" "Mouser"
+		(property "Supplier 2" ""
 			(at 231.648 181.61 0)
 			(hide yes)
@@
 					(size 1.27 1.27)
 				)
-			)
-		)
-		(property "Supplier 3" "JLCPCB"
-			(at 187.96 180.34 0)
-			(hide yes)
-			(show_name no)
-			(do_not_autoplace no)
-			(effects
-				(font
-					(size 1.27 1.27)
-				)
-				(justify left)
-			)
-		)
-		(property "Supplier Part Num 3" "C5277086"
-			(at 190.5 180.34 0)
-			(hide yes)
-			(show_name no)
-			(do_not_autoplace no)
-			(effects
-				(font
-					(size 1.27 1.27)
-				)
-				(justify left)
-			)
-		)
-		(property "Label" "LABEL"
-			(at 193.04 180.34 0)
-			(hide yes)
-			(show_name no)
-			(do_not_autoplace no)
-			(effects
-				(font
-					(size 1.27 1.27)
-				)
-				(justify left)
-			)
-		)
-		(property "JLCPCB Part Num" "C5277086"
-			(at 195.58 180.34 0)
-			(hide yes)
-			(show_name no)
-			(do_not_autoplace no)
-			(effects
-				(font
-					(size 1.27 1.27)
-				)
-				(justify left)
 			)
 		)
@@
 	)
 	(symbol
-		(lib_id "BR_Virtual_Parts:TP_SQUARE_TH_1mm")
+		(lib_id "BR_Virtual_Parts:TP_SQUARE_TH_2mm")
 		(at 238.76 185.42 90)
 		(unit 1)
 		(body_style 1)
-		(exclude_from_sim yes)
+		(exclude_from_sim no)
 		(in_bom no)
 		(on_board yes)
@@
 			)
 		)
-		(property "Footprint" "BR_Virtual_Parts:TP_SQUARE_TH_1mm"
+		(property "Footprint" "BR_Virtual_Parts:TP_SQUARE_TH_2mm"
 			(at 231.394 184.15 0)
 			(hide yes)
@@
 			)
 		)
-		(property "Datasheet" "https://wmsc.lcsc.com/wmsc/upload/file/pdf/v2/lcsc/2307040929_ronghe-RH-5000_C5277086.pdf"
+		(property "Datasheet" ""
 			(at 231.267 185.166 0)
 			(hide yes)
@@
 			)
 		)
-		(property "Description" "test pad through hole"
+		(property "Description" "test pad, through hole"
 			(at 238.76 185.42 0)
 			(hide yes)
@@
 			)
 		)
-		(property "Manufacturer" "ronghe"
+		(property "Manufacturer" ""
 			(at 230.759 186.944 0)
 			(hide yes)
@@
 			)
 		)
-		(property "Manufacturer Part Num" "RH-5000"
+		(property "Manufacturer Part Num" ""
 			(at 231.648 185.674 0)
 			(hide yes)
@@
 			)
 		)
-		(property "BRE Number" "BRE-000074"
-			(at 175.26 185.42 0)
-			(hide yes)
-			(show_name no)
-			(do_not_autoplace no)
-			(effects
-				(font
-					(size 1.27 1.27)
-				)
-				(justify left)
-			)
-		)
-		(property "Supplier 1" "DigiKey"
+		(property "Supplier 1" ""
 			(at 231.14 187.325 0)
 			(hide yes)
@@
 			)
 		)
-		(property "Supplier 2" "Mouser"
+		(property "Supplier 2" ""
 			(at 231.648 186.69 0)
 			(hide yes)
@@
 			)
 		)
-		(property "Supplier 3" "JLCPCB"
-			(at 187.96 185.42 0)
-			(hide yes)
-			(show_name no)
-			(do_not_autoplace no)
-			(effects
-				(font
-					(size 1.27 1.27)
-				)
-				(justify left)
-			)
-		)
-		(property "Supplier Part Num 3" "C5277086"
-			(at 190.5 185.42 0)
-			(hide yes)
-			(show_name no)
-			(do_not_autoplace no)
-			(effects
-				(font
-					(size 1.27 1.27)
-				)
-				(justify left)
-			)
-		)
-		(property "Label" "LABEL"
-			(at 193.04 185.42 0)
-			(hide yes)
-			(show_name no)
-			(do_not_autoplace no)
-			(effects
-				(font
-					(size 1.27 1.27)
-				)
-				(justify left)
-			)
-		)
-		(property "JLCPCB Part Num" "C5277086"
-			(at 195.58 185.42 0)
-			(hide yes)
-			(show_name no)
-			(do_not_autoplace no)
-			(effects
-				(font
-					(size 1.27 1.27)
-				)
-				(justify left)
-			)
-		)
