File: MCU.kicad_sch (KiCad schematic)
At the start: 103 parts, among them J301 LABEL, J302 LABEL, U301 STM32H563AII3Q, X301 25MHz 8pF

Commit message: more work
Parts:
- renumbered C303 to C301, C304 to C302, C302 to C303, C307 to C304, C311 to C305, C312 to C306, C301 to C307, C313 to C308, C314 to C309, C315 to C310, C305 to C311, C306 to C312, C317 to C313, C318 to C314, C319 to C315, C308 to C316, C320 to C317, C321 to C318, C322 to C319, C309 to C320, C310 to C321, C323 to C322, C324 to C323, C325 to C324, C316 to C325, J302 to J301, J301 to J302, R111 to R303, R112 to R305, R305 to R306, TP302 to TP301, TP303 to TP302, TP306 to TP303, TP305 to TP304, TP307 to TP305, TP308 to TP306, TP358 to TP307, TP309 to TP308, TP317 to TP309, TP318 to TP310, TP310 to TP311, TP311 to TP312, TP312 to TP313, TP313 to TP314, TP314 to TP315, TP315 to TP316, TP316 to TP317, TP319 to TP318, TP320 to TP319, TP321 to TP320, TP301 to TP321, TP365 to TP330, TP330 to TP331, TP331 to TP332, TP332 to TP333, TP333 to TP334, TP367 to TP335, TP334 to TP336, TP335 to TP337, TP336 to TP338, TP337 to TP339, TP338 to TP340, TP339 to TP341, TP340 to TP342, TP341 to TP343, TP342 to TP344, TP343 to TP345, TP344 to TP346, TP345 to TP347, TP346 to TP348, TP347 to TP349, TP348 to TP350, TP349 to TP351, TP350 to TP352, TP351 to TP353, TP352 to TP354, TP353 to TP355, TP354 to TP356, TP355 to TP357, TP356 to TP358, TP357 to TP359, TP366 to TP360, TP304 to TP361, TP359 to TP362, TP360 to TP363, TP361 to TP364, TP362 to TP365, TP363 to TP366, TP364 to TP367

Commit message: more work
Connections:
- net PHY_REF_CLK renamed MAC.REF_CLK
- no-connect marks 66 -> 67
Changed lines of the file:
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@@
 	(text "AF11: ETH_RMII_REF_CLK"
 		(exclude_from_sim no)
-		(at 305.308 168.656 0)
+		(at 289.306 168.656 0)
 		(effects
 			(font
@@
 	)
 	(junction
-		(at 256.54 167.64)
-		(diameter 0)
-		(color 0 0 0 0)
-	)
-	(junction
 		(at 132.08 259.08)
 		(diameter 0)
@@
 	)
 	(no_connect
+		(at 231.14 345.44)
+	)
+	(no_connect
 		(at 231.14 279.4)
 	)
@@
 	(wire
 		(pts
-			(xy 256.54 167.64) (xy 266.7 167.64)
-		)
-		(stroke
-			(width 0)
-			(type default)
-		)
-	)
-	(wire
-		(pts
 			(xy 231.14 332.74) (xy 256.54 332.74)
 		)
@@
 		)
 	)
+	(label "MAC.REF_CLK"
+		(at 256.54 274.32 180)
+		(effects
+			(font
+				(size 1.27 1.27)
+			)
+			(justify right bottom)
+		)
+	)
 	(label "MAC.CRSDV"
 		(at 256.54 182.88 180)
@@
 		)
 	)
-	(label "PHY_REF_CLK"
-		(at 256.54 274.32 180)
-		(effects
-			(font
-				(size 1.27 1.27)
-			)
-			(justify right bottom)
-		)
-	)
 	(label "TX_EN"
 		(at 248.92 299.72 0)
@@
 		)
 	)
-	(hierarchical_label "PHY_REF_CLK"
-		(shape output)
-		(at 266.7 167.64 0)
-		(effects
-			(font
-				(size 1.27 1.27)
-			)
-			(justify left)
-		)
-	)

Commit message: more work
Parts:
- removed J301, J302: LABEL, BR_Connectors:PinHeader_1x02_P2.54mm_Vertical, symbol BR_Connectors_Header:Header_Pin_01x02_2.54mm_Vert_PTH
- R303, R305: footprint BR_Passives:R_0201_0603Metric-minimized -> BR_Passives:C_0402_1005Metric-minimized; symbol BR_Resistors_0201:R_0201_10k -> BR_Resistors_0402:R_0402_10k; BRE Number BRE-000261 -> BRE-000292; JLCPCB Part Num C106225 -> C144807; Manufacturer Part Num RC0201FR-0710KL -> AC0402FR-0710KL; Supplier 2 Mouser -> DigiKey; Supplier Part Num 1 311-10.0KMCT-ND -> YAG3436CT-ND; Supplier Part Num 2 603-RC0201FR-0710KL -> YAG3436TR-ND; Supplier Part Num 3 C106225 -> C144807

Commit message: more work
Parts:
- added TP368, TP369, TP370: TP_ROUND_TH_300um, BR_Virtual_Parts:TP_ROUND_SMT_300um, symbol BR_Virtual_Parts:TP_ROUND_SMT_300um
Connections:
- net FDCAN2.TX: now reaches U301.C6 (PB6)
- net FDCAN2.TX: now also TP368.1
- net GPIO_C8: now reaches U301.E9 (PC8)
- net GPIO_C8: now also TP370.1
- net FDCAN2.RX: now reaches U301.H9 (PD9)
- net FDCAN2.RX: now also TP369.1
- no-connect marks 67 -> 64

Commit message: fixing some errors
Parts:
- R303, R304, R305, R306: footprint BR_Passives:C_0402_1005Metric-minimized -> BR_Passives:R_0402_1005Metric-minimized
Changed lines of the file:
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@@
 			)
 		)
-		(property "Footprint" "BR_Passives:C_0402_1005Metric-minimized"
+		(property "Footprint" "BR_Passives:R_0402_1005Metric-minimized"
 			(at 302.26 17.78 0)
 			(hide yes)
@@
 			)
 		)
-		(property "Footprint" "BR_Passives:C_0402_1005Metric-minimized"
+		(property "Footprint" "BR_Passives:R_0402_1005Metric-minimized"
 			(at 292.1 17.78 0)
 			(hide yes)
@@
 			)
 		)
-		(property "Footprint" "BR_Passives:C_0402_1005Metric-minimized"
+		(property "Footprint" "BR_Passives:R_0402_1005Metric-minimized"
 			(at 292.1 -5.08 0)
 			(hide yes)
@@
 			)
 		)
-		(property "Footprint" "BR_Passives:C_0402_1005Metric-minimized"
+		(property "Footprint" "BR_Passives:R_0402_1005Metric-minimized"
 			(at 302.26 -5.08 0)
 			(hide yes)

Commit message: more cleanup
Other:
- note added: "AF9: FDCAN2_RX"
- note added: "AF9: FDCAN2_TX"
- note removed: "AF11: ETH_MDC"
- note removed: "AF3: TIM8_CH2"
Changed lines of the file:
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@@
 	(generator_version "10.0")
 	(paper "A2")
-	(text "AF11: ETH_MDC"
-		(exclude_from_sim no)
-		(at 280.67 178.816 0)
-		(effects
-			(font
-				(size 1.27 1.27)
-			)
-			(justify right bottom)
-		)
-	)
 	(text "AF11: ETH_RMII_REF_CLK"
 		(exclude_from_sim no)
@@
 		)
 	)
-	(text "GPIO"
-		(exclude_from_sim no)
-		(at 105.664 188.976 0)
-		(effects
-			(font
-				(size 1.27 1.27)
-			)
-			(justify left bottom)
-		)
-	)
 	(text "AF11: ETH_RMII_TXD0"
 		(exclude_from_sim no)
@@
 		)
 	)
-	(text "GPIO"
-		(exclude_from_sim no)
-		(at 101.854 194.056 0)
-		(effects
-			(font
-				(size 1.27 1.27)
-			)
-			(justify left bottom)
-		)
-	)
 	(text "AF4: I2C1_SCL"
 		(exclude_from_sim no)
@@
 		)
 	)
-	(text "GPIO"
-		(exclude_from_sim no)
-		(at 104.902 186.436 0)
-		(effects
-			(font
-				(size 1.27 1.27)
-			)
-			(justify left bottom)
-		)
-	)
 	(text "AF5: SPI5_SCK"
 		(exclude_from_sim no)
@@
 		)
 	)
-	(text "GPIO"
-		(exclude_from_sim no)
-		(at 101.854 196.596 0)
-		(effects
-			(font
-				(size 1.27 1.27)
-			)
-			(justify left bottom)
-		)
-	)
 	(text "AF11: ETH_RMII_TX_EN"
 		(exclude_from_sim no)
@@
 		)
 	)
-	(text "GPIO"
-		(exclude_from_sim no)
-		(at 101.6 201.676 0)
-		(effects
-			(font
-				(size 1.27 1.27)
-			)
-			(justify left bottom)
-		)
-	)
 	(text "AF9: OCTOSPI1_CLK"
 		(exclude_from_sim no)
@@
 	(text "AF10: OCTOSPI1_IO3"
 		(exclude_from_sim no)
-		(at 104.14 305.816 0)
+		(at 102.87 305.816 0)
 		(effects
 			(font
@@
 		)
 	)
-	(text "AF3: TIM8_CH2"
-		(exclude_from_sim no)
-		(at 278.638 270.256 0)
-		(effects
-			(font
-				(size 1.27 1.27)
-			)
-			(justify left bottom)
-		)
-	)
 	(text "AF4: I2C1_SDA"
 		(exclude_from_sim no)
@@
 	(text "AF10: OCTOSPI1_IO0"
 		(exclude_from_sim no)
-		(at 104.14 310.896 0)
+		(at 102.87 310.896 0)
 		(effects
 			(font
@@
 	(text "AF10: OCTOSPI1_IO1"
 		(exclude_from_sim no)
-		(at 104.14 313.436 0)
+		(at 102.87 313.436 0)
 		(effects
 			(font
@@
 		)
 	)
+	(text "AF9: FDCAN2_TX"
+		(exclude_from_sim no)
+		(at 282.448 224.536 0)
+		(effects
+			(font
+				(size 1.27 1.27)
+			)
+			(justify right bottom)
+		)
+	)
 	(text "AF10: OCTOSPI1_IO6\n"
 		(exclude_from_sim no)
@@
 		)
 	)
+	(text "AF9: FDCAN2_RX"
+		(exclude_from_sim no)
+		(at 281.94 318.516 0)
+		(effects
+			(font
+				(size 1.27 1.27)
+			)
+			(justify right bottom)
+		)
+	)
 	(text "AF3: TIM8_CH1"
 		(exclude_from_sim no)
-		(at 93.726 199.136 0)
+		(at 97.79 199.136 0)
 		(effects
 			(font
@@
 	(wire
 		(pts
-			(xy 256.54 180.34) (xy 266.7 180.34)
+			(xy 256.54 180.34) (xy 267.97 180.34)
 		)
 		(stroke
@@
 		)
 	)
-	(label "ADC2_INP2"
+	(label "RX_SIG"
 		(at 133.35 322.58 0)
 		(effects
@@
 		)
 	)
+	(label "V_SENSE"
+		(at 133.35 317.5 0)
+		(effects
+			(font
+				(size 1.27 1.27)
+			)
+			(justify left bottom)
+		)
+	)
 	(label "OCTOSPI1.IO2"
 		(at 256.54 342.9 180)
@@
 		)
 	)
-	(label "GPIO_D4"
+	(label "TX_DAMP"
 		(at 256.54 304.8 180)
 		(effects
@@
 	(hierarchical_label "ADC12_INP3"
 		(shape input)
-		(at 266.7 180.34 0)
+		(at 267.97 180.34 0)
 		(effects
 			(font

Commit message: clearing ERC errors and some ref des tidy up
Other:
- note added: "DEBUG_LED"
- note added: "MOTOR_DIR"
- note added: "MOTOR_EN"
- note added: "MOTOR_MODE0"
- note added: "MOTOR_MODE1"
- note added: "MOTOR_STEP"
- note added: "MOTOR_VREF"
- note added: "MOTOR_nFAULT"
- note added: "MOTOR_nSLEEP"
- note added: "PHY_nRST"
- note added: "RX_SIG"
- note added: "TGC_RST"
- note added: "TX_DAMP"
- note added: "TX_DSD"
- note added: "TX_EN"
- note added: "TX_I_SENSE"
- note added: "TX_PWM_A"
- note added: "TX_PWM_B"
- note added: "TX_SIG"
- note added: "VTX_EN"
- note added: "VTX_SENSE"
- note added: "V_SENSE"
- note added: "V_THERM"
