File: vrx_boost.kicad_sch (KiCad schematic)
At the start: 12 parts, among them U1301 LM27313XMFX/NOPB

Commit message: work
Parts:
- removed TP1301, TP1302: TP_RING_TH, BR_Connectors:TEST-TH_BD2.54-P1.4_RED, symbol BR_Connectors:TP_Ring_PTH
Other:
- moved on the sheet: C1301, C1302, C1303, D1301, L1301, NT1301, R1301, R1302, R1303, U1301

Commit message: getting really close to final
Parts:
- R1301, R1302, R1303: footprint BR_Passives:C_0402_1005Metric-minimized -> BR_Passives:R_0402_1005Metric-minimized
Changed lines of the file:
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@@
 			)
 		)
-		(property "Footprint" "BR_Passives:C_0402_1005Metric-minimized"
+		(property "Footprint" "BR_Passives:R_0402_1005Metric-minimized"
 			(at 256.54 116.84 0)
 			(hide yes)
@@
 			)
 		)
-		(property "Footprint" "BR_Passives:C_0402_1005Metric-minimized"
+		(property "Footprint" "BR_Passives:R_0402_1005Metric-minimized"
 			(at 287.02 135.89 0)
 			(hide yes)
@@
 			)
 		)
-		(property "Footprint" "BR_Passives:C_0402_1005Metric-minimized"
+		(property "Footprint" "BR_Passives:R_0402_1005Metric-minimized"
 			(at 219.71 198.12 0)
 			(hide yes)

Commit message: clearing ERC errors and some ref des tidy up
Parts:
- C1303: value 10uF 10V -> 10uF 35V; footprint BR_Passives:C_0402_1005Metric-minimized -> BR_Passives:C_0603_1608Metric-minimized; symbol BR_Capacitors_0402:C_0402_10uF_10V_X5R_20% -> BR_Capacitors_0603:C_0603_10uF_35V_X5R_20%; BRE Number BRE-000015 -> BRE-001305; JLCPCB Part Num C315248 -> C49326366; Manufacturer Samsung Electro-Mechanics -> AIDE CAPACITOR; Manufacturer Part Num CL05A106MP5NUNC -> 0603X5R106M350NT; Supplier 1 DigiKey -> (none); Supplier 2 Mouser -> (none); Supplier 3 JLCPCB -> (none); Supplier Part Num 1 1276-1450-6-ND -> (none); Supplier Part Num 2 187-CL05A106MP5NUNC -> (none); Supplier Part Num 3 C315248 -> (none)
Other:
- note added: "Vin = 5V Vout = 11V Vout = Vin/(1-D) -> D = 56.5% (including diode drop 0.5V) -> F = 1.6 MHz -> tON = 353ns"
- note removed: "Vin = 5V Vout = 7V Vout = Vin/(1-D) -> D = 31.5% (including diode drop) -> tON = 197ns"
Changed lines of the file:
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@@
 		)
 	)
-	(text "Vin = 5V\nVout = 7V\nVout = Vin/(1-D)\n-> D = 31.5% (including diode drop)\n-> tON = 197ns"
+	(text "Vin = 5V\nVout = 11V\nVout = Vin/(1-D)\n-> D = 56.5% (including diode drop 0.5V)\n-> F = 1.6 MHz\n-> tON = 353ns"
 		(exclude_from_sim no)
 		(at 205.994 151.892 0)
@@
 	)
 	(symbol
-		(lib_id "BR_Capacitors_0402:C_0402_10uF_10V_X5R_20%")
+		(lib_id "BR_Capacitors_0603:C_0603_10uF_35V_X5R_20%")
 		(at 320.04 212.09 0)
 		(unit 1)
@@
 			)
 		)
-		(property "Value" "10uF 10V"
+		(property "Value" "10uF 35V"
 			(at 322.58 213.3662 0)
 			(show_name no)
@@
 			)
 		)
-		(property "Footprint" "BR_Passives:C_0402_1005Metric-minimized"
+		(property "Footprint" "BR_Passives:C_0603_1608Metric-minimized"
 			(at 320.04 135.89 0)
 			(hide yes)
@@
 			)
 		)
-		(property "Datasheet" "https://mm.digikey.com/Volume0/opasdata/d220001/medias/docus/2614/CL05A106MP5NUNC_Spec.pdf"
+		(property "Datasheet" "https://www.lcsc.com/datasheet/C49326366.pdf"
 			(at 320.04 138.43 0)
 			(hide yes)
@@
 			)
 		)
-		(property "Description" "10uF 10V X5R 20% Ceramic Capacitor 0402"
+		(property "Description" "10uF 35V X5R20% Ceramic Capacitor 0603"
 			(at 320.04 140.97 0)
 			(hide yes)
@@
 			)
 		)
-		(property "Manufacturer" "Samsung Electro-Mechanics"
+		(property "Manufacturer" "AIDE CAPACITOR"
 			(at 320.04 143.51 0)
 			(hide yes)
@@
 			)
 		)
-		(property "Manufacturer Part Num" "CL05A106MP5NUNC"
+		(property "Manufacturer Part Num" "0603X5R106M350NT"
 			(at 320.04 146.05 0)
 			(hide yes)
@@
 			)
 		)
-		(property "BRE Number" "BRE-000015"
+		(property "BRE Number" "BRE-001305"
 			(at 320.04 148.59 0)
 			(hide yes)
@@
 			)
 		)
-		(property "Supplier 1" "DigiKey"
+		(property "JLCPCB Part Num" "C49326366"
 			(at 320.04 151.13 0)
 			(hide yes)
 			(show_name no)
-			(do_not_autoplace no)
-			(effects
-				(font
-					(size 1.27 1.27)
-				)
-				(justify left)
-			)
-		)
-		(property "Supplier 2" "Mouser"
-			(at 320.04 153.67 0)
-			(hide yes)
-			(show_name no)
-			(do_not_autoplace no)
-			(effects
-				(font
-					(size 1.27 1.27)
-				)
-				(justify left)
-			)
-		)
-		(property "Supplier 3" "JLCPCB"
-			(at 320.04 156.21 0)
-			(hide yes)
-			(show_name no)
-			(do_not_autoplace no)
-			(effects
-				(font
-					(size 1.27 1.27)
-				)
-				(justify left)
-			)
-		)
-		(property "Supplier Part Num 1" "1276-1450-6-ND"
-			(at 320.04 158.75 0)
-			(hide yes)
-			(show_name no)
-			(do_not_autoplace no)
-			(effects
-				(font
-					(size 1.27 1.27)
-				)
-				(justify left)
-			)
-		)
-		(property "Supplier Part Num 2" "187-CL05A106MP5NUNC"
-			(at 320.04 161.29 0)
-			(hide yes)
-			(show_name no)
-			(do_not_autoplace no)
-			(effects
-				(font
-					(size 1.27 1.27)
-				)
-				(justify left)
-			)
-		)
-		(property "Supplier Part Num 3" "C315248"
-			(at 320.04 163.83 0)
-			(hide yes)
-			(show_name no)
-			(do_not_autoplace no)
-			(effects
-				(font
-					(size 1.27 1.27)
-				)
-				(justify left)
-			)
-		)
-		(property "JLCPCB Part Num" "C315248"
-			(at 320.04 166.37 0)
-			(hide yes)
-			(show_name no)
