File: power-layouts/sonar-dev-board-power-layouts.kicad_pcb (KiCad board)
At the start: 6 copper layers, 480.1 x 265.6 mm, 379 parts, among them J1001 TX_OUT_GAIN, J101 POWER, J102 DEBUG, J103 PORT1, J104 FPGA, J105 ETHERNET, J106 SYNC, J107 SONAR+, J108 SONAR+, J109 SONAR-, J110 SONAR-, J111 TRANSDUCER, J112 MOTOR, J1201 RFBT, J1202 RDAC, J401 RX_IN, J402 PREAMP, J403 BIAS_RES, J404 BIAS_RES, J405 GAIN_RES, J406 LPF_CAP, J407 VARAMP_OUT, J501 LABEL, J502 LABEL, J601 CAP, J901 OCTOSPI, Q101 DMP6023LSS-13, Q1201 SQJ974EP, Q1501 MMBT3904L, Q1503 MMBT3904L, T101 B65655B0010X000, T701 HR641680E, U1001 SL9062D, U1002 LT1794, U1003 CSA230PASOT235, U101 LIS2DH12TR, U1101 TLV62569DBVR, U1201 LM5122MHX/NOPB, U1202 DAC53401DSGR, U1301 LM27313XMFX/NOPB, U1401 MG78L05T3, U1501 EPC23104ENGRT, U1502 EPC23104ENGRT, U1601 DRV8426RGER, U301 STM32H563AII3Q, U401 MD0100DK6-G, U402 OPA1612AIDR, U403 AD8338ACPZ-R7, U404 WS72552M-8/TR, U601 DAC53401DSGR, U602 DAC53401DSGR, U603 74LVC1G66GW,125, U701 DP83825IRMQR, U801 MIC28517T-E/PHA, U901 S27KL0642DPBHB023, X301 25MHz 8pF

Commit message: Update sonar-dev-board-power-layouts.kicad_pcb
Routing:
- net /TX/VCC_AB: track 31.5 -> 97.2 mm
- net /TX/GND_AB: track 94.1 -> 156.2 mm
- net /TX/2X_ATT_AB: track 0.00 -> 48.6 mm
- net GND: track 304.3 -> 337.6 mm, vias 48 -> 50
- net /TX/TX_EN_AB: track 0.00 -> 31.3 mm
- net /TX/10X_ATT_AB: track 0.00 -> 28.2 mm
- net /TX/SIG_IN_AB: track 4.04 -> 24.7 mm
- net /TX/SIG_OUT+_AB: track 18.3 -> 14.9 mm

Commit message: Update sonar-dev-board-power-layouts.kicad_pcb
Routing:
- net VCC: track 37.7 -> 60.0 mm, vias 40 -> 42
- net /TX/TX_EN_AB: track 31.3 -> 32.2 mm
Changed lines of the file:
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@@
+	)
+	(segment
+		(start 489.61 -101.88)
+		(end 489.61 -104.11)
+		(width 0.1)
+		(layer "F.Cu")
+		(net 69)
+	)
+	(segment
+		(start 507.39 -103.61)
+		(end 506.5 -104.5)
+		(width 0.1)
+		(layer "F.Cu")
+		(net 69)
 	)
 	(segment
@@
 	)
 	(segment
+		(start 489.61 -104.11)
+		(end 490 -104.5)
+		(width 0.1)
+		(layer "F.Cu")
+		(net 69)
+	)
+	(segment
 		(start 507.39 -101.88)
 		(end 507.39 -97.71)
@@
 		(start 420 -36.619)
 		(end 420 -37)
+		(width 0.1)
+		(layer "F.Cu")
+		(net 69)
+	)
+	(segment
+		(start 507.39 -101.88)
+		(end 507.39 -103.61)
 		(width 0.1)
 		(layer "F.Cu")
@@
 	)
 	(via
+		(at 490 -104.5)
+		(size 0.6)
+		(drill 0.3)
+		(layers "F.Cu" "B.Cu")
+		(net 69)
+	)
+	(via
 		(at 194.405 -59.855)
 		(size 0.6)
@@
 	)
 	(via
+		(at 506.5 -104.5)
+		(size 0.6)
+		(drill 0.3)
+		(layers "F.Cu" "B.Cu")
+		(net 69)
+	)
+	(via
 		(at 193.135 -62.903)
 		(size 0.6)
@@
 		(drill 0.3)
 		(layers "F.Cu" "B.Cu")
+		(net 69)
+	)
+	(segment
+		(start 490 -104.5)
+		(end 506.5 -104.5)
+		(width 0.1)
+		(layer "B.Cu")
 		(net 69)
 	)
@@
 	)
 	(segment
+		(start 497.934 -109.136)
+		(end 499.77 -107.3)
+		(width 0.1)
+		(layer "F.Cu")
+		(net 139)
+	)
+	(segment
+		(start 488 -103)
+		(end 488 -104.5)
+		(width 0.1)
+		(layer "F.Cu")
+		(net 139)
+	)
+	(segment
+		(start 491.389 -106.389)
+		(end 491.389 -109.136)
+		(width 0.1)
+		(layer "F.Cu")
+		(net 139)
+	)
+	(segment
+		(start 490.464 -105.464)
+		(end 491.389 -106.389)
+		(width 0.1)
+		(layer "F.Cu")
+		(net 139)
+	)
+	(segment
 		(start 487.831 -102.831)
+		(end 488 -103)
+		(width 0.1)
+		(layer "F.Cu")
+		(net 139)
+	)
+	(segment
+		(start 486.325 -89.055)
 		(end 487.831 -90.561)
 		(width 0.1)
@@
 	)
 	(segment
-		(start 491.389 -106.389)
+		(start 488 -104.5)
+		(end 488.964 -105.464)
+		(width 0.1)
+		(layer "F.Cu")
+		(net 139)
+	)
+	(segment
+		(start 491.389 -109.136)
+		(end 497.934 -109.136)
+		(width 0.1)
+		(layer "F.Cu")
+		(net 139)
+	)
+	(segment
+		(start 487.831 -90.561)
 		(end 487.831 -102.831)
 		(width 0.1)
@@
 	)
 	(segment
-		(start 491.389 -109.136)
-		(end 491.389 -106.389)
-		(width 0.1)
-		(layer "F.Cu")
-		(net 139)
-	)
-	(segment
-		(start 487.831 -90.561)
-		(end 486.325 -89.055)
-		(width 0.1)
-		(layer "F.Cu")
-		(net 139)
-	)
-	(segment
-		(start 499.77 -107.3)
-		(end 497.934 -109.136)
-		(width 0.1)
-		(layer "F.Cu")
-		(net 139)
-	)
-	(segment
-		(start 497.934 -109.136)
-		(end 491.389 -109.136)
-		(width 0.1)
-		(layer "F.Cu")
+		(start 488.964 -105.464)
+		(end 490.464 -105.464)
+		(width 0.1)
+		(layer "F.Cu")

Commit message: Update sonar-dev-board-power-layouts.kicad_pcb
Parts:
- moved J501 51.9 mm to (449.5, -87.6)
- moved J502 51.9 mm to (449.5, -78.0)
- moved R501 51.9 mm to (439.6, -70.6)
- moved R502 51.9 mm to (439.8, -72.3)
- moved TP501 51.9 mm to (437.3, -72.1)
- moved TP502 51.9 mm to (437.3, -69.8)
- moved TP503 51.9 mm to (437.3, -67.5)
- moved TP504 51.9 mm to (437.3, -65.2)
- moved C1501 40.5 mm to (458.4, -57.4)
- moved C1502 40.5 mm to (451.4, -57.1)
- moved C1503 40.5 mm to (456.9, -55.4)
- moved C1504 40.5 mm to (446.3, -55.4)
- moved C1505 40.5 mm to (440.9, -57.2)
- moved C1506 40.5 mm to (447.9, -57.3)
- moved NT1501 40.5 mm to (449.3, -52.4)
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